Commit message: gazebo quase 100%

File: build/hand_pack/urdf/combined_robot.urdf.xacro (robot description, xacro)
@@ -1 +1 @@
-/home/biolab-linux/RoboticArm/src/hand_pack/urdf/combined_robot.urdf.xacro
+/home/lucas-pc/RoboticArm/src/hand_pack/urdf/combined_robot.urdf.xacro

File: build/hand_pack/urdf/hand.xacro (robot description, xacro)
@@ -1 +1 @@
-/home/biolab-linux/RoboticArm/src/hand_pack/urdf/hand.xacro
+/home/lucas-pc/RoboticArm/src/hand_pack/urdf/hand.xacro

File: build/hand_pack/urdf/hj_hand_gazebo.xacro (robot description, xacro)
@@ -1 +1 @@
-/home/biolab-linux/RoboticArm/src/hand_pack/urdf/hj_hand_gazebo.xacro
+/home/lucas-pc/RoboticArm/src/hand_pack/urdf/hj_hand_gazebo.xacro

File: build/hand_pack/urdf/hj_hand_transmission.xacro (robot description, xacro)
@@ -1 +1 @@
-/home/biolab-linux/RoboticArm/src/hand_pack/urdf/hj_hand_transmission.xacro
+/home/lucas-pc/RoboticArm/src/hand_pack/urdf/hj_hand_transmission.xacro

File: build/hand_pack/urdf/hj_hand_world.urdf.xacro (robot description, xacro)
@@ -1 +1 @@
-/home/biolab-linux/RoboticArm/src/hand_pack/urdf/hj_hand_world.urdf.xacro
+/home/lucas-pc/RoboticArm/src/hand_pack/urdf/hj_hand_world.urdf.xacro

File: install/hand_pack/share/hand_pack/urdf/hand.xacro (robot description, xacro)
@@ -437,5 +437,5 @@
             </visual>
             <inertial>
-                  <mass value="0.001"/>
+                  <mass value="0.1"/>
                   <inertia ixx="1.0e-03" ixy="0.0" ixz="0.0"
                iyy="1.0e-03" iyz="0.0"
@@ -491,5 +491,5 @@
             </visual>
             <inertial>
-                  <mass value="0.001"/>
+                  <mass value="0.1"/>
                   <inertia ixx="1.0e-03" ixy="0.0" ixz="0.0"
                iyy="1.0e-03" iyz="0.0"
@@ -1050,5 +1050,5 @@
             </visual>
             <inertial>
-                  <mass value="0.001"/>
+                  <mass value="0.1"/>
                   <inertia ixx="1.0e-03" ixy="0.0" ixz="0.0"
                iyy="1.0e-03" iyz="0.0"
@@ -1104,5 +1104,5 @@
             </visual>
             <inertial>
-                  <mass value="0.001"/>
+                  <mass value="0.1"/>
                   <inertia ixx="1.0e-03" ixy="0.0" ixz="0.0"
                iyy="1.0e-03" iyz="0.0"
@@ -1158,5 +1158,5 @@
             </visual>
             <inertial>
-                  <mass value="0.001"/>
+                  <mass value="0.1"/>
                   <inertia ixx="1.0e-03" ixy="0.0" ixz="0.0"
                iyy="1.0e-03" iyz="0.0"
@@ -1212,5 +1212,5 @@
             </visual>
             <inertial>
-                  <mass value="0.001"/>
+                  <mass value="0.1"/>
                   <inertia ixx="1.0e-03" ixy="0.0" ixz="0.0"
                iyy="1.0e-03" iyz="0.0"

File: install/ur_description/share/ur_description/urdf/inc/ur_common.xacro (robot description, xacro)
@@ -1 +1 @@
-/home/biolab-linux/RoboticArm/src/ur_description/urdf/inc/ur_common.xacro
+/home/lucas-pc/RoboticArm/src/ur_description/urdf/inc/ur_common.xacro

File: install/ur_description/share/ur_description/urdf/inc/ur_joint_control.xacro (robot description, xacro)
@@ -1 +1 @@
-/home/biolab-linux/RoboticArm/src/ur_description/urdf/inc/ur_joint_control.xacro
+/home/lucas-pc/RoboticArm/src/ur_description/urdf/inc/ur_joint_control.xacro

File: install/ur_description/share/ur_description/urdf/inc/ur_sensors.xacro (robot description, xacro)
@@ -1 +1 @@
-/home/biolab-linux/RoboticArm/src/ur_description/urdf/inc/ur_sensors.xacro
+/home/lucas-pc/RoboticArm/src/ur_description/urdf/inc/ur_sensors.xacro

File: install/ur_description/share/ur_description/urdf/inc/ur_transmissions.xacro (robot description, xacro)
@@ -1 +1 @@
-/home/biolab-linux/RoboticArm/src/ur_description/urdf/inc/ur_transmissions.xacro
+/home/lucas-pc/RoboticArm/src/ur_description/urdf/inc/ur_transmissions.xacro

File: install/ur_description/share/ur_description/urdf/ros2_control_mock_hardware.xacro (robot description, xacro)
@@ -1 +1 @@
-/home/biolab-linux/RoboticArm/src/ur_description/urdf/ros2_control_mock_hardware.xacro
+/home/lucas-pc/RoboticArm/src/ur_description/urdf/ros2_control_mock_hardware.xacro

File: install/ur_description/share/ur_description/urdf/ur.urdf.xacro (robot description, xacro)
@@ -1 +1 @@
-/home/biolab-linux/RoboticArm/src/ur_description/urdf/ur.urdf.xacro
+/home/lucas-pc/RoboticArm/src/ur_description/urdf/ur.urdf.xacro

File: install/ur_description/share/ur_description/urdf/ur_macro.xacro (robot description, xacro)
@@ -1 +1 @@
-/home/biolab-linux/RoboticArm/src/ur_description/urdf/ur_macro.xacro
+/home/lucas-pc/RoboticArm/src/ur_description/urdf/ur_macro.xacro

File: install/ur_description/share/ur_description/urdf/ur_mocked.urdf.xacro (robot description, xacro)
@@ -1 +1 @@
-/home/biolab-linux/RoboticArm/src/ur_description/urdf/ur_mocked.urdf.xacro
+/home/lucas-pc/RoboticArm/src/ur_description/urdf/ur_mocked.urdf.xacro

File: src/ur_description/urdf/ur.urdf.xacro (robot description, xacro)
@@ -2,10 +2,10 @@
 <robot xmlns:xacro="http://wiki.ros.org/xacro" name="$(arg name)">
    <!-- robot name parameter -->
-   <xacro:arg name="name" default="ur5"/>
+   <xacro:arg name="name" default="ur"/>
    <!-- import main macro -->
    <xacro:include filename="$(find ur_description)/urdf/ur_macro.xacro"/>
    <!-- possible 'ur_type' values: ur3, ur3e, ur5, ur5e, ur10, ur10e, ur16e, ur20, ur30 -->
    <!-- the default value should raise an error in case this was called without defining the type -->
-   <xacro:arg name="ur5" default="ur5"/>
+   <xacro:arg name="ur_type" default="ur5x"/>
    <!-- parameters -->
    <xacro:arg name="tf_prefix" default="" />
@@ -18,5 +18,5 @@
    <xacro:arg name="safety_pos_margin" default="0.15"/>
    <xacro:arg name="safety_k_position" default="20"/>
-   <!--When using  simulations absolute paths are necessary.-->
+   <!--When using gazebo simulations absolute paths are necessary.-->
    <xacro:arg name="force_abs_paths" default="false" />
    <!-- create link fixed to the "world" -->

File: src/ur_description/urdf/ur_mocked.urdf.xacro (robot description, xacro)
@@ -2,5 +2,5 @@
 <robot xmlns:xacro="http://wiki.ros.org/xacro" name="$(arg name)">
   <!-- robot name parameter -->
-  <xacro:arg name="name" default="ur5"/>
+  <xacro:arg name="name" default="ur"/>
   <!-- import main macro -->
   <xacro:include filename="$(find ur_description)/urdf/ur_macro.xacro"/>
@@ -8,5 +8,5 @@
   <!-- possible 'ur_type' values: ur3, ur3e, ur5, ur5e, ur10, ur10e, ur16e, ur20, ur30 -->
   <!-- the default value should raise an error in case this was called without defining the type -->
-  <xacro:arg name="ur5" default="ur5"/>
+  <xacro:arg name="ur_type" default="ur5x"/>
   <!-- parameters -->
   <xacro:arg name="tf_prefix" default="" />
