Commit message: testes

File: src/hand_pack/urdf/hand.xacro (robot description, xacro)
@@ -4,5 +4,5 @@
         <visual>
             <geometry>
-                <box size="0.01 0.10 0.01"/> <!-- Ajuste conforme necessário -->
+                <box size="0.001 0.001 0.001"/>
             </geometry>
             <material name="white">
