Commit message: integração CR10 + COVVI: lançamento Gazebo/RViz, GUI combinada e limpeza do gitignore
Remove build/install/log/DOBOT do rastreamento git; adiciona launch files CR10+COVVI, combined_gui, world factory e configs de controladores.

File: src/hand_pack/urdf/linear_covvi_hand_gazebo.urdf (robot description, URDF)
Before this commit: robot covvi_digital_twin_perfect, 87 links, 86 joints
Links:
- link base_link: geometry collision box size=0.08 0.08 0.08; visual mesh filename=package://hand_pack/urdf/linear_meshes/right_base_link.STL scale=0.001 0.001 0.001
- link index_distal: geometry collision mesh filename=package://hand_pack/urdf/linear_meshes/right_index_distal.S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 scale=0.001 0.001 0.001; visual mesh filename=package://hand_pack/urdf/linear_meshes/right_index_distal.S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 scale=0.001 0.001 0.001
- link index_follower: geometry collision mesh filename=package://hand_pack/urdf/linear_meshes/right_index_follower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 scale=0.001 0.001 0.001; visual mesh filename=package://hand_pack/urdf/linear_meshes/right_index_follower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 scale=0.001 0.001 0.001
- link index_knuckle: geometry collision mesh filename=package://hand_pack/urdf/linear_meshes/right_index_knuckle.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 scale=0.001 0.001 0.001; visual mesh filename=package://hand_pack/urdf/linear_meshes/right_index_knuckle.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 scale=0.001 0.001 0.001
- link index_link: geometry collision mesh filename=package://hand_pack/urdf/linear_meshes/right_index_link.STL scale=0.001 0.001 0.001; visual mesh filename=package://hand_pack/urdf/linear_meshes/right_index_link.STL scale=0.001 0.001 0.001
- link index_proximal: geometry collision mesh filename=package://hand_pack/urdf/linear_meshes/right_index_proximal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 scale=0.001 0.001 0.001; visual mesh filename=package://hand_pack/urdf/linear_meshes/right_index_proximal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 scale=0.001 0.001 0.001
- link lisa: geometry collision mesh filename=package://hand_pack/urdf/linear_meshes/right_lisa.STL scale=0.001 0.001 0.001; visual mesh filename=package://hand_pack/urdf/linear_meshes/right_lisa.STL scale=0.001 0.001 0.001
- link little_distal: geometry collision mesh filename=package://hand_pack/urdf/linear_meshes/right_little_distal.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 scale=0.001 0.001 0.001; visual mesh filename=package://hand_pack/urdf/linear_meshes/right_little_distal.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 scale=0.001 0.001 0.001
- link little_follower: geometry collision mesh filename=package://hand_pack/urdf/linear_meshes/right_little_followe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 scale=0.001 0.001 0.001; visual mesh filename=package://hand_pack/urdf/linear_meshes/right_little_followe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 scale=0.001 0.001 0.001
- link little_knuckle: geometry collision mesh filename=package://hand_pack/urdf/linear_meshes/right_little_knuckle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 scale=0.001 0.001 0.001; visual mesh filename=package://hand_pack/urdf/linear_meshes/right_little_knuckle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 scale=0.001 0.001 0.001
- link little_link: geometry collision mesh filename=package://hand_pack/urdf/linear_meshes/right_little_link.STL scale=0.001 0.001 0.001; visual mesh filename=package://hand_pack/urdf/linear_meshes/right_little_link.STL scale=0.001 0.001 0.001
- link little_proximal: geometry collision mesh filename=package://hand_pack/urdf/linear_meshes/right_little_proxima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 scale=0.001 0.001 0.001; visual mesh filename=package://hand_pack/urdf/linear_meshes/right_little_proxima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 scale=0.001 0.001 0.001
- link middle_distal: geometry collision mesh filename=package://hand_pack/urdf/linear_meshes/right_middle_distal.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 scale=0.001 0.001 0.001; visual mesh filename=package://hand_pack/urdf/linear_meshes/right_middle_distal.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 scale=0.001 0.001 0.001
- link middle_follower: geometry collision mesh filename=package://hand_pack/urdf/linear_meshes/right_middle_followe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 scale=0.001 0.001 0.001; visual mesh filename=package://hand_pack/urdf/linear_meshes/right_middle_followe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 scale=0.001 0.001 0.001
- link middle_knuckle: geometry collision mesh filename=package://hand_pack/urdf/linear_meshes/right_middle_knuckle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 scale=0.001 0.001 0.001; visual mesh filename=package://hand_pack/urdf/linear_meshes/right_middle_knuckle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 scale=0.001 0.001 0.001
- link middle_link: geometry collision mesh filename=package://hand_pack/urdf/linear_meshes/right_middle_link.STL scale=0.001 0.001 0.001; visual mesh filename=package://hand_pack/urdf/linear_meshes/right_middle_link.STL scale=0.001 0.001 0.001
- link middle_proximal: geometry collision mesh filename=package://hand_pack/urdf/linear_meshes/right_middle_proxima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 scale=0.001 0.001 0.001; visual mesh filename=package://hand_pack/urdf/linear_meshes/right_middle_proxima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 scale=0.001 0.001 0.001
- link ring_distal: geometry collision mesh filename=package://hand_pack/urdf/linear_meshes/right_ring_distal.STL scale=0.001 0.001 0.001; visual mesh filename=package://hand_pack/urdf/linear_meshes/right_ring_distal.STL scale=0.001 0.001 0.001
- link ring_follower: geometry collision mesh filename=package://hand_pack/urdf/linear_meshes/right_ring_follower.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 scale=0.001 0.001 0.001; visual mesh filename=package://hand_pack/urdf/linear_meshes/right_ring_follower.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 scale=0.001 0.001 0.001
- link ring_knuckle: geometry collision mesh filename=package://hand_pack/urdf/linear_meshes/right_ring_knuckle.S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 scale=0.001 0.001 0.001; visual mesh filename=package://hand_pack/urdf/linear_meshes/right_ring_knuckle.S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 scale=0.001 0.001 0.001
- link ring_link: geometry collision mesh filename=package://hand_pack/urdf/linear_meshes/right_ring_link.STL scale=0.001 0.001 0.001; visual mesh filename=package://hand_pack/urdf/linear_meshes/right_ring_link.STL scale=0.001 0.001 0.001
- link ring_proximal: geometry collision mesh filename=package://hand_pack/urdf/linear_meshes/right_ring_proximal.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 scale=0.001 0.001 0.001; visual mesh filename=package://hand_pack/urdf/linear_meshes/right_ring_proximal.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 scale=0.001 0.001 0.001
- link thumb_chassis: geometry collision mesh filename=package://hand_pack/urdf/linear_meshes/right_thumb_chassis.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 scale=0.001 0.001 0.001; visual mesh filename=package://hand_pack/urdf/linear_meshes/right_thumb_chassis.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 scale=0.001 0.001 0.001
- link thumb_distal: geometry collision mesh filename=package://hand_pack/urdf/linear_meshes/right_thumb_distal.S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 scale=0.001 0.001 0.001; visual mesh filename=package://hand_pack/urdf/linear_meshes/right_thumb_distal.S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 scale=0.001 0.001 0.001
- link thumb_follower: geometry collision mesh filename=package://hand_pack/urdf/linear_meshes/right_thumb_follower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 scale=0.001 0.001 0.001; visual mesh filename=package://hand_pack/urdf/linear_meshes/right_thumb_follower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 scale=0.001 0.001 0.001
- link thumb_link: geometry collision mesh filename=package://hand_pack/urdf/linear_meshes/right_thumb_link.STL scale=0.001 0.001 0.001; visual mesh filename=package://hand_pack/urdf/linear_meshes/right_thumb_link.STL scale=0.001 0.001 0.001
- link thumb_proximal: geometry collision mesh filename=package://hand_pack/urdf/linear_meshes/right_thumb_proximal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 scale=0.001 0.001 0.001; visual mesh filename=package://hand_pack/urdf/linear_meshes/right_thumb_proximal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 scale=0.001 0.001 0.001
Joints:
- joint Index: limit lower=0.00000000000000000000 upper=1.00000000000000000000 effort=10.0 velocity=1.0 -> lower=0.00000000000000000000 upper=1.60000000000000008882 effort=10.0 velocity=1.0
- joint Little: limit lower=0.00000000000000000000 upper=1.00000000000000000000 effort=10.0 velocity=1.0 -> lower=0.00000000000000000000 upper=1.60000000000000008882 effort=10.0 velocity=1.0
- joint Middle: limit lower=0.00000000000000000000 upper=1.00000000000000000000 effort=10.0 velocity=1.0 -> lower=0.00000000000000000000 upper=1.60000000000000008882 effort=10.0 velocity=1.0
- joint Ring: limit lower=0.00000000000000000000 upper=1.00000000000000000000 effort=10.0 velocity=1.0 -> lower=0.00000000000000000000 upper=1.60000000000000008882 effort=10.0 velocity=1.0
- joint Thumb: limit lower=0.00000000000000000000 upper=1.00000000000000000000 effort=10.0 velocity=1.0 -> lower=0.00000000000000000000 upper=1.60000000000000008882 effort=10.0 velocity=1.0
- joint _index_distal_j01: limit lower=0.00000002107342395030 upper=1.33574110944277979485 effort=10.0 velocity=1.0 -> lower=0.00000002107342395030 upper=2.13718576246439351252 effort=10.0 velocity=1.0
- joint _index_distal_j_index_distal: origin xyz=-1.5070534999285634 -7.578488986309617 1.0647940483682832 rpy=-0.00000002107342395030 0 0 -> xyz=-0.02411285599885701347 -0.12125582378095388358 0.01703670477389252966 rpy=-0.00000002107342395030 0 0
- joint _index_distal_j_input_joint: origin xyz=1.5070534999285634 7.578488986309617 -1.0647940483682832 rpy=-0.00000002107342395030 0 0 -> xyz=0.02411285599885701347 0.12125582378095388358 -0.01703670477389252966 rpy=-0.00000002107342395030 0 0
- joint _index_follower_j01: limit lower=-0.00000000000000005551 upper=0.26422627443923901724 effort=10.0 velocity=1.0 -> lower=-0.00000000000000005551 upper=0.42276203910278248310 effort=10.0 velocity=1.0
- joint _index_follower_j_index_follower: origin xyz=-1.3289578043144759 -4.198973084070179 1.3040394900270869 rpy=0.00000000000000005551 0 0 -> xyz=-0.02126332486903161414 -0.06718356934512285938 0.02086463184043339109 rpy=0.00000000000000005551 0 0
- joint _index_follower_j_input_joint: origin xyz=1.3289578043144759 4.198973084070179 -1.3040394900270869 rpy=0.00000000000000005551 0 0 -> xyz=0.02126332486903161414 0.06718356934512285938 -0.02086463184043339109 rpy=0.00000000000000005551 0 0
- joint _index_knuckle_j01: limit lower=0.00000002107342400581 upper=1.25181521906792703192 effort=10.0 velocity=1.0 -> lower=0.00000002107342400581 upper=2.00290433786462918064 effort=10.0 velocity=1.0
- joint _index_knuckle_j_index_knuckle: origin xyz=-1.366060538694307 -5.324288335618494 1.4862338867796852 rpy=-0.00000002107342400581 0 0 -> xyz=-0.02185696861910891090 -0.08518861336989590194 0.02377974218847496435 rpy=-0.00000002107342400581 0 0
- joint _index_knuckle_j_input_joint: origin xyz=1.366060538694307 5.324288335618494 -1.4862338867796852 rpy=-0.00000002107342400581 0 0 -> xyz=0.02185696861910891090 0.08518861336989590194 -0.02377974218847496435 rpy=-0.00000002107342400581 0 0
- joint _index_link_j01: limit lower=-0.00000000000000033307 upper=1.33574038782547499515 effort=10.0 velocity=1.0 -> lower=-0.00000000000000033307 upper=2.13718462052076008106 effort=10.0 velocity=1.0; type fixed -> revolute
- joint _index_link_j_index_link: origin xyz=-1.3943596383310624 -5.7976159675856795 1.1863715383108244 rpy=0.00000000000000033307 0 0 -> xyz=-0.02230975421329699920 -0.09276185548137087789 0.01898194461297319016 rpy=0.00000000000000033307 0 0
- joint _index_link_j_input_joint: origin xyz=1.3943596383310624 5.7976159675856795 -1.1863715383108244 rpy=0.00000000000000033307 0 0 -> xyz=0.02230975421329699920 0.09276185548137087789 -0.01898194461297319016 rpy=0.00000000000000033307 0 0
- joint _index_proximal_j01: limit lower=0.00000001490116086078 upper=1.51604341403629772067 effort=10.0 velocity=1.0 -> lower=0.00000001490116086078 upper=2.42566945351737972558 effort=10.0 velocity=1.0
- joint _index_proximal_j_index_proximal: origin xyz=-1.4438636714684971 -5.709859526571508 0.9223736237943079 rpy=-0.00000001490116086078 0 0 -> xyz=-0.02310181874349595543 -0.09135775242514412864 0.01475797798070892577 rpy=-0.00000001490116086078 0 0
- joint _index_proximal_j_input_joint: origin xyz=1.4438636714684971 5.709859526571508 -0.9223736237943079 rpy=-0.00000001490116086078 0 0 -> xyz=0.02310181874349595543 0.09135775242514412864 -0.01475797798070892577 rpy=-0.00000001490116086078 0 0
- joint _lisa_j_input_joint: origin xyz=0.6649580028042494 1.243265013263121 0.7747941474098129 rpy=-0.00000001490116097180 0 0 -> xyz=0.01063932804486799125 0.01989224021220993913 0.01239670635855700739 rpy=-0.00000001490116097180 0 0
- joint _lisa_j_lisa: origin xyz=-0.6649580028042494 -1.243265013263121 -0.7747941474098129 rpy=-0.00000001490116097180 0 0 -> xyz=-0.01063932804486799125 -0.01989224021220993913 -0.01239670635855700739 rpy=-0.00000001490116097180 0 0
- joint _little_distal_j01: limit lower=0.00000001490116086078 upper=1.31664154360936347388 effort=10.0 velocity=1.0 -> lower=0.00000001490116086078 upper=2.10662646083428528598 effort=10.0 velocity=1.0
- joint _little_distal_j_input_joint: origin xyz=-2.2520633889913793 6.742798507484316 -0.4576241639059808 rpy=-0.00000001490116086078 0 0 -> xyz=-0.03603301422386206987 0.10788477611974905956 -0.00732198662249569296 rpy=-0.00000001490116086078 0 0
- joint _little_distal_j_little_distal: origin xyz=2.2520633889913793 -6.742798507484316 0.4576241639059808 rpy=-0.00000001490116086078 0 0 -> xyz=0.03603301422386206987 -0.10788477611974905956 0.00732198662249569296 rpy=-0.00000001490116086078 0 0
- joint _little_follower_j01: limit lower=-0.00000000000000005551 upper=0.26422625333146310123 effort=10.0 velocity=1.0 -> lower=-0.00000000000000005551 upper=0.42276200533034102857 effort=10.0 velocity=1.0
- joint _little_follower_j_input_joint: origin xyz=-1.9684499144753422 3.76508855610884 -0.6557183186033343 rpy=0.00000000000000005551 0 0 -> xyz=-0.03149519863160547828 0.06024141689774143577 -0.01049149309765334825 rpy=0.00000000000000005551 0 0
- joint _little_follower_j_little_follower: origin xyz=1.9684499144753422 -3.76508855610884 0.6557183186033343 rpy=0.00000000000000005551 0 0 -> xyz=0.03149519863160547828 -0.06024141689774143577 0.01049149309765334825 rpy=0.00000000000000005551 0 0
- joint _little_knuckle_j01: limit lower=0.00000001490116097180 upper=1.25181530552105346743 effort=10.0 velocity=1.0 -> lower=0.00000001490116097180 upper=2.00290447989298892040 effort=10.0 velocity=1.0
- joint _little_knuckle_j_input_joint: origin xyz=-2.120049770560409 4.884666340842449 -0.8121441650432416 rpy=-0.00000001490116097180 0 0 -> xyz=-0.03392079632896654456 0.07815466145347918503 -0.01299430664069186649 rpy=-0.00000001490116097180 0 0
- joint _little_knuckle_j_little_knuckle: origin xyz=2.120049770560409 -4.884666340842449 0.8121441650432416 rpy=-0.00000001490116097180 0 0 -> xyz=0.03392079632896654456 -0.07815466145347918503 0.01299430664069186649 rpy=-0.00000001490116097180 0 0
- joint _little_link_j01: limit lower=-0.00000000000000022204 upper=1.31664159359669952210 effort=10.0 velocity=1.0 -> lower=-0.00000000000000022204 upper=2.10662654975471985708 effort=10.0 velocity=1.0; type fixed -> revolute
- joint _little_link_j_input_joint: origin xyz=-2.1349977455383624 5.35345561586718 -0.5047965951115416 rpy=0.00000000000000022204 0 0 -> xyz=-0.03415996392861379849 0.08565528985387488303 -0.00807674552178466558 rpy=0.00000000000000022204 0 0
- joint _little_link_j_little_link: origin xyz=2.1349977455383624 -5.35345561586718 0.5047965951115416 rpy=0.00000000000000022204 0 0 -> xyz=0.03415996392861379849 -0.08565528985387488303 0.00807674552178466558 rpy=0.00000000000000022204 0 0
- joint _little_proximal_j01: limit lower=-0.00000000000000022204 upper=1.51604353824540583062 effort=10.0 velocity=1.0 -> lower=-0.00000000000000022204 upper=2.42566966119265003954 effort=10.0 velocity=1.0
- joint _little_proximal_j_input_joint: origin xyz=-2.057319724224253 5.270538765035208 -0.24661281778517774 rpy=0.00000000000000022204 0 0 -> xyz=-0.03291711558758805140 0.08432862024056332617 -0.00394580508456284385 rpy=0.00000000000000022204 0 0
- joint _little_proximal_j_little_proximal: origin xyz=2.057319724224253 -5.270538765035208 0.24661281778517774 rpy=0.00000000000000022204 0 0 -> xyz=0.03291711558758805140 -0.08432862024056332617 0.00394580508456284385 rpy=0.00000000000000022204 0 0
- joint _middle_distal_j01: limit lower=0.00000002107342389479 upper=1.34986013639683699594 effort=10.0 velocity=1.0 -> lower=0.00000002107342389479 upper=2.15977620559088512309 effort=10.0 velocity=1.0
- joint _middle_distal_j_input_joint: origin xyz=0.19688874055412953 8.022176691106141 -1.0461525552984252 rpy=-0.00000002107342389479 0 0 -> xyz=0.00315021984886607260 0.12835482705769826750 -0.01673844088477480230 rpy=-0.00000002107342389479 0 0
- joint _middle_distal_j_middle_distal: origin xyz=-0.19688874055412953 -8.022176691106141 1.0461525552984252 rpy=-0.00000002107342389479 0 0 -> xyz=-0.00315021984886607260 -0.12835482705769826750 0.01673844088477480230 rpy=-0.00000002107342389479 0 0
- joint _middle_follower_j01: limit lower=-0.00000000000000005551 upper=0.26422641895880316643 effort=10.0 velocity=1.0 -> lower=-0.00000000000000005551 upper=0.42276227033408514400 effort=10.0 velocity=1.0
- joint _middle_follower_j_input_joint: origin xyz=0.15980891875989833 4.386421938486642 -1.361995902128741 rpy=0.00000000000000005551 0 0 -> xyz=0.00255694270015837354 0.07018275101578626274 -0.02179193443405985989 rpy=0.00000000000000005551 0 0
- joint _middle_follower_j_middle_follower: origin xyz=-0.15980891875989833 -4.386421938486642 1.361995902128741 rpy=0.00000000000000005551 0 0 -> xyz=-0.00255694270015837354 -0.07018275101578626274 0.02179193443405985989 rpy=0.00000000000000005551 0 0
- joint _middle_knuckle_j01: limit lower=-0.00000000000000022204 upper=1.25181499257524886382 effort=10.0 velocity=1.0 -> lower=-0.00000000000000022204 upper=2.00290398812039871501 effort=10.0 velocity=1.0
- joint _middle_knuckle_j_input_joint: origin xyz=0.1327026701136127 5.513391010636881 -1.535525341148929 rpy=0.00000000000000022204 0 0 -> xyz=0.00212324272181780302 0.08821425617019010290 -0.02456840545838286441 rpy=0.00000000000000022204 0 0
- joint _middle_knuckle_j_middle_knuckle: origin xyz=-0.1327026701136127 -5.513391010636881 1.535525341148929 rpy=0.00000000000000022204 0 0 -> xyz=-0.00212324272181780302 -0.08821425617019010290 0.02456840545838286441 rpy=0.00000000000000022204 0 0
- joint _middle_link_j01: limit lower=-0.00000000000000027756 upper=1.34986028913700639720 effort=10.0 velocity=1.0 -> lower=-0.00000000000000027756 upper=2.15977646261921041315 effort=10.0 velocity=1.0; type fixed -> revolute
- joint _middle_link_j_input_joint: origin xyz=0.1485688418916027 5.985445071198181 -1.232930729247692 rpy=0.00000000000000027756 0 0 -> xyz=0.00237710147026564322 0.09576712113917089375 -0.01972689166796307361 rpy=0.00000000000000027756 0 0
- joint _middle_link_j_middle_link: origin xyz=-0.1485688418916027 -5.985445071198181 1.232930729247692 rpy=0.00000000000000027756 0 0 -> xyz=-0.00237710147026564322 -0.09576712113917089375 0.01972689166796307361 rpy=0.00000000000000027756 0 0
- joint _middle_proximal_j01: limit lower=-0.00000000000000055511 upper=1.51604368978712988891 effort=10.0 velocity=1.0 -> lower=-0.00000000000000055511 upper=2.42566990365940826635 effort=10.0 velocity=1.0
- joint _middle_proximal_j_input_joint: origin xyz=0.20973618604014632 5.898534205707262 -0.9712659363241443 rpy=0.00000000000000055511 0 0 -> xyz=0.00335577897664234102 0.09437654729131618458 -0.01554025498118630916 rpy=0.00000000000000055511 0 0
- joint _middle_proximal_j_middle_proximal: origin xyz=-0.20973618604014632 -5.898534205707262 0.9712659363241443 rpy=0.00000000000000055511 0 0 -> xyz=-0.00335577897664234102 -0.09437654729131618458 0.01554025498118630916 rpy=0.00000000000000055511 0 0
- joint _ring_distal_j01: limit lower=-0.00000000000000033307 upper=1.34878317629562749502 effort=10.0 velocity=1.0 -> lower=-0.00000000000000033307 upper=2.15805308207300416967 effort=10.0 velocity=1.0
- joint _ring_distal_j_input_joint: origin xyz=-1.1013923470306217 7.892249906746441 -0.8122495227348061 rpy=0.00000000000000033307 0 0 -> xyz=-0.01762227755248994832 0.12627599850794304914 -0.01299599236375689748 rpy=0.00000000000000033307 0 0
- joint _ring_distal_j_ring_distal: origin xyz=1.1013923470306217 -7.892249906746441 0.8122495227348061 rpy=0.00000000000000033307 0 0 -> xyz=0.01762227755248994832 -0.12627599850794304914 0.01299599236375689748 rpy=0.00000000000000033307 0 0
- joint _ring_follower_j01: limit lower=-0.00000000000000005551 upper=0.26423062522385393214 effort=10.0 velocity=1.0 -> lower=-0.00000000000000005551 upper=0.42276900035816633583 effort=10.0 velocity=1.0
- joint _ring_follower_j_input_joint: origin xyz=-1.0102042572973156 4.387462722072228 -1.078451840885562 rpy=0.00000000000000005551 0 0 -> xyz=-0.01616326811675704994 0.07019940355315565372 -0.01725522945416899101 rpy=0.00000000000000005551 0 0
- joint _ring_follower_j_ring_follower: origin xyz=1.0102042572973156 -4.387462722072228 1.078451840885562 rpy=0.00000000000000005551 0 0 -> xyz=0.01616326811675704994 -0.07019940355315565372 0.01725522945416899101 rpy=0.00000000000000005551 0 0
- joint _ring_knuckle_j01: limit lower=-0.00000000000000033307 upper=1.25181510906761417345 effort=10.0 velocity=1.0 -> lower=-0.00000000000000033307 upper=2.00290417450818303280 effort=10.0 velocity=1.0
- joint _ring_knuckle_j_input_joint: origin xyz=-1.076287437386446 5.513612382054195 -1.2467379346586647 rpy=0.00000000000000033307 0 0 -> xyz=-0.01722059899818313700 0.08821779811286711848 -0.01994780695453863412 rpy=0.00000000000000033307 0 0
- joint _ring_knuckle_j_ring_knuckle: origin xyz=1.076287437386446 -5.513612382054195 1.2467379346586647 rpy=0.00000000000000033307 0 0 -> xyz=0.01722059899818313700 -0.08821779811286711848 0.01994780695453863412 rpy=0.00000000000000033307 0 0
- joint _ring_link_j01: limit lower=-0.00000000000000027756 upper=1.34878364034376607705 effort=10.0 velocity=1.0 -> lower=-0.00000000000000027756 upper=2.15805382455002581210 effort=10.0 velocity=1.0; type fixed -> revolute
- joint _ring_link_j_input_joint: origin xyz=-1.078572100240299 5.984454531834645 -0.9417015242120699 rpy=0.00000000000000027756 0 0 -> xyz=-0.01725715360384478397 0.09575127250935432099 -0.01506722438739311817 rpy=0.00000000000000027756 0 0
- joint _ring_link_j_ring_link: origin xyz=1.078572100240299 -5.984454531834645 0.9417015242120699 rpy=0.00000000000000027756 0 0 -> xyz=0.01725715360384478397 -0.09575127250935432099 0.01506722438739311817 rpy=0.00000000000000027756 0 0
- joint _ring_proximal_j01: limit lower=-0.00000000000000022204 upper=1.51604328762193540925 effort=10.0 velocity=1.0 -> lower=-0.00000000000000022204 upper=2.42566926019509709889 effort=10.0 velocity=1.0
- joint _ring_proximal_j_input_joint: origin xyz=-1.0126493534897856 5.898556410085637 -0.6806766424213684 rpy=0.00000000000000022204 0 0 -> xyz=-0.01620238965583657015 0.09437690256137018507 -0.01089082627874189517 rpy=0.00000000000000022204 0 0
- joint _ring_proximal_j_ring_proximal: origin xyz=1.0126493534897856 -5.898556410085637 0.6806766424213684 rpy=0.00000000000000022204 0 0 -> xyz=0.01620238965583657015 -0.09437690256137018507 0.01089082627874189517 rpy=0.00000000000000022204 0 0
- joint _thumb_chassis_j_input_joint: origin xyz=1.514903298568658 1.432445559291959 0.7844313794953435 rpy=-0.00000002107342389479 0 0 -> xyz=0.02423845277709852850 0.02291912894867134329 0.01255090207192549601 rpy=-0.00000002107342389479 0 0
- joint _thumb_chassis_j_thumb_chassis: origin xyz=-1.514903298568658 -1.432445559291959 -0.7844313794953435 rpy=-0.00000002107342389479 0 0 -> xyz=-0.02423845277709852850 -0.02291912894867134329 -0.01255090207192549601 rpy=-0.00000002107342389479 0 0
- joint _thumb_distal_j01: limit lower=-0.00000000000000033307 upper=1.06686018440504426508 effort=10.0 velocity=1.0 -> lower=-0.00000000000000033307 upper=1.70697629504807113499 effort=10.0 velocity=1.0
- joint _thumb_distal_j_input_joint: origin xyz=5.380329672338689 4.204299673061814 0.6377162617521437 rpy=0.00000000000000033307 0 0 -> xyz=0.08608527475741903356 0.06726879476898903198 0.01020346018803429920 rpy=0.00000000000000033307 0 0
- joint _thumb_distal_j_thumb_distal: origin xyz=-5.380329672338689 -4.204299673061814 -0.6377162617521437 rpy=0.00000000000000033307 0 0 -> xyz=-0.08608527475741903356 -0.06726879476898903198 -0.01020346018803429920 rpy=0.00000000000000033307 0 0
- joint _thumb_follower_j01: limit lower=-0.00000000000000022204 upper=0.93732763826281428887 effort=10.0 velocity=1.0 -> lower=-0.00000000000000022204 upper=1.49972422122050308424 effort=10.0 velocity=1.0
- joint _thumb_follower_j_input_joint: origin xyz=2.720835809921482 2.848104079083896 0.8664653479863773 rpy=0.00000000000000022204 0 0 -> xyz=0.04353337295874371016 0.04556966526534234063 0.01386344556778203695 rpy=0.00000000000000022204 0 0
- joint _thumb_follower_j_thumb_follower: origin xyz=-2.720835809921482 -2.848104079083896 -0.8664653479863773 rpy=0.00000000000000022204 0 0 -> xyz=-0.04353337295874371016 -0.04556966526534234063 -0.01386344556778203695 rpy=0.00000000000000022204 0 0
- joint _thumb_link_j01: limit lower=-0.00000000000000016653 upper=0.76799454671461697686 effort=10.0 velocity=1.0 -> lower=-0.00000000000000016653 upper=1.22879127474338734061 effort=10.0 velocity=1.0
- joint _thumb_link_j_input_joint: origin xyz=2.3175473087185097 1.6154584748791998 0.7720019170415124 rpy=0.00000000000000016653 0 0 -> xyz=0.03708075693949615392 0.02584733559806719899 0.01235203067266419860 rpy=0.00000000000000016653 0 0
- joint _thumb_link_j_thumb_link: origin xyz=-2.3175473087185097 -1.6154584748791998 -0.7720019170415124 rpy=0.00000000000000016653 0 0 -> xyz=-0.03708075693949615392 -0.02584733559806719899 -0.01235203067266419860 rpy=0.00000000000000016653 0 0
- joint _thumb_proximal_j01: limit lower=-0.00000000000000016653 upper=0.72022188617106019937 effort=10.0 velocity=1.0 -> lower=-0.00000000000000016653 upper=1.15235501787369631899 effort=10.0 velocity=1.0
- joint _thumb_proximal_j_input_joint: origin xyz=2.8720356292446443 1.353914565668949 0.6504721331635288 rpy=0.00000000000000016653 0 0 -> xyz=0.04595257006791431120 0.02166263305070318529 0.01040755413061646151 rpy=0.00000000000000016653 0 0
- joint _thumb_proximal_j_thumb_proximal: origin xyz=-2.8720356292446443 -1.353914565668949 -0.6504721331635288 rpy=0.00000000000000016653 0 0 -> xyz=-0.04595257006791431120 -0.02166263305070318529 -0.01040755413061646151 rpy=0.00000000000000016653 0 0
