Commit message: grip corrigido

File: src/hand_pack/urdf/linear_covvi_hand_gazebo.urdf (robot description, URDF)
Before this commit: robot covvi_digital_twin_perfect, 87 links, 86 joints
Links:
- link index_distal: geometry collision box size=0.0166 0.0380 0.0275; visual mesh filename=package://hand_pack/urdf/linear_meshes/right_index_distal.S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 scale=0.001 0.001 0.001
- link index_proximal: geometry collision box size=0.0145 0.0425 0.0205; visual mesh filename=package://hand_pack/urdf/linear_meshes/right_index_proximal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 scale=0.001 0.001 0.001
- link little_distal: geometry collision box size=0.0161 0.0293 0.0254; visual mesh filename=package://hand_pack/urdf/linear_meshes/right_little_distal.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 scale=0.001 0.001 0.001
- link little_proximal: geometry collision box size=0.0143 0.0367 0.0179; visual mesh filename=package://hand_pack/urdf/linear_meshes/right_little_proxima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 scale=0.001 0.001 0.001
- link middle_distal: geometry collision box size=0.0172 0.0378 0.0289; visual mesh filename=package://hand_pack/urdf/linear_meshes/right_middle_distal.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 scale=0.001 0.001 0.001
- link middle_proximal: geometry collision box size=0.0146 0.0461 0.0207; visual mesh filename=package://hand_pack/urdf/linear_meshes/right_middle_proxima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 scale=0.001 0.001 0.001
- link ring_distal: geometry collision box size=0.0158 0.0379 0.0278; visual mesh filename=package://hand_pack/urdf/linear_meshes/right_ring_distal.STL scale=0.001 0.001 0.001
- link ring_proximal: geometry collision box size=0.0144 0.0444 0.0206; visual mesh filename=package://hand_pack/urdf/linear_meshes/right_ring_proximal.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 scale=0.001 0.001 0.001
- link thumb_distal: geometry collision box size=0.0324 0.0332 0.0210; visual mesh filename=package://hand_pack/urdf/linear_meshes/right_thumb_distal.S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 scale=0.001 0.001 0.001
- link thumb_proximal: geometry collision box size=0.0485 0.0537 0.0216; visual mesh filename=package://hand_pack/urdf/linear_meshes/right_thumb_proximal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 scale=0.001 0.001 0.001
Joints:
- joint Index: limit lower=0.00000000000000000000 upper=1.60000000000000008882 effort=10.0 velocity=1.0 -> lower=0.00000000000000000000 upper=1.60000000000000008882 effort=1.0 velocity=1.0
- joint Little: limit lower=0.00000000000000000000 upper=1.60000000000000008882 effort=10.0 velocity=1.0 -> lower=0.00000000000000000000 upper=1.60000000000000008882 effort=1.0 velocity=1.0
- joint Middle: limit lower=0.00000000000000000000 upper=1.60000000000000008882 effort=10.0 velocity=1.0 -> lower=0.00000000000000000000 upper=1.60000000000000008882 effort=1.0 velocity=1.0
- joint Ring: limit lower=0.00000000000000000000 upper=1.60000000000000008882 effort=10.0 velocity=1.0 -> lower=0.00000000000000000000 upper=1.60000000000000008882 effort=1.0 velocity=1.0
- joint Rotate: limit lower=0.00000000000000000000 upper=1.00000000000000000000 effort=10.0 velocity=1.0 -> lower=0.00000000000000000000 upper=1.00000000000000000000 effort=1.0 velocity=1.0
- joint Thumb: limit lower=0.00000000000000000000 upper=1.60000000000000008882 effort=10.0 velocity=1.0 -> lower=0.00000000000000000000 upper=1.60000000000000008882 effort=1.0 velocity=1.0
- joint _index_distal_j01: limit lower=0.00000002107342395030 upper=2.13718576246439351252 effort=10.0 velocity=1.0 -> lower=0.00000002107342395030 upper=2.13718576246439351252 effort=1.0 velocity=1.0
- joint _index_follower_j01: limit lower=-0.00000000000000005551 upper=0.42276203910278248310 effort=10.0 velocity=1.0 -> lower=-0.00000000000000005551 upper=0.42276203910278248310 effort=1.0 velocity=1.0
- joint _index_knuckle_j01: limit lower=0.00000002107342400581 upper=2.00290433786462918064 effort=10.0 velocity=1.0 -> lower=0.00000002107342400581 upper=2.00290433786462918064 effort=1.0 velocity=1.0
- joint _index_link_j01: limit lower=-0.00000000000000033307 upper=2.13718462052076008106 effort=10.0 velocity=1.0 -> lower=-0.00000000000000033307 upper=2.13718462052076008106 effort=1.0 velocity=1.0
- joint _index_proximal_j01: limit lower=0.00000001490116086078 upper=2.42566945351737972558 effort=10.0 velocity=1.0 -> lower=0.00000001490116086078 upper=2.42566945351737972558 effort=1.0 velocity=1.0
- joint _lisa_j01: limit lower=0.00000001490116097180 upper=1.07337743464992829701 effort=10.0 velocity=1.0 -> lower=0.00000001490116097180 upper=1.07337743464992829701 effort=1.0 velocity=1.0
- joint _little_distal_j01: limit lower=0.00000001490116086078 upper=2.10662646083428528598 effort=10.0 velocity=1.0 -> lower=0.00000001490116086078 upper=2.10662646083428528598 effort=1.0 velocity=1.0
- joint _little_follower_j01: limit lower=-0.00000000000000005551 upper=0.42276200533034102857 effort=10.0 velocity=1.0 -> lower=-0.00000000000000005551 upper=0.42276200533034102857 effort=1.0 velocity=1.0
- joint _little_knuckle_j01: limit lower=0.00000001490116097180 upper=2.00290447989298892040 effort=10.0 velocity=1.0 -> lower=0.00000001490116097180 upper=2.00290447989298892040 effort=1.0 velocity=1.0
- joint _little_link_j01: limit lower=-0.00000000000000022204 upper=2.10662654975471985708 effort=10.0 velocity=1.0 -> lower=-0.00000000000000022204 upper=2.10662654975471985708 effort=1.0 velocity=1.0
- joint _little_proximal_j01: limit lower=-0.00000000000000022204 upper=2.42566966119265003954 effort=10.0 velocity=1.0 -> lower=-0.00000000000000022204 upper=2.42566966119265003954 effort=1.0 velocity=1.0
- joint _middle_distal_j01: limit lower=0.00000002107342389479 upper=2.15977620559088512309 effort=10.0 velocity=1.0 -> lower=0.00000002107342389479 upper=2.15977620559088512309 effort=1.0 velocity=1.0
- joint _middle_follower_j01: limit lower=-0.00000000000000005551 upper=0.42276227033408514400 effort=10.0 velocity=1.0 -> lower=-0.00000000000000005551 upper=0.42276227033408514400 effort=1.0 velocity=1.0
- joint _middle_knuckle_j01: limit lower=-0.00000000000000022204 upper=2.00290398812039871501 effort=10.0 velocity=1.0 -> lower=-0.00000000000000022204 upper=2.00290398812039871501 effort=1.0 velocity=1.0
- joint _middle_link_j01: limit lower=-0.00000000000000027756 upper=2.15977646261921041315 effort=10.0 velocity=1.0 -> lower=-0.00000000000000027756 upper=2.15977646261921041315 effort=1.0 velocity=1.0
- joint _middle_proximal_j01: limit lower=-0.00000000000000055511 upper=2.42566990365940826635 effort=10.0 velocity=1.0 -> lower=-0.00000000000000055511 upper=2.42566990365940826635 effort=1.0 velocity=1.0
- joint _ring_distal_j01: limit lower=-0.00000000000000033307 upper=2.15805308207300416967 effort=10.0 velocity=1.0 -> lower=-0.00000000000000033307 upper=2.15805308207300416967 effort=1.0 velocity=1.0
- joint _ring_follower_j01: limit lower=-0.00000000000000005551 upper=0.42276900035816633583 effort=10.0 velocity=1.0 -> lower=-0.00000000000000005551 upper=0.42276900035816633583 effort=1.0 velocity=1.0
- joint _ring_knuckle_j01: limit lower=-0.00000000000000033307 upper=2.00290417450818303280 effort=10.0 velocity=1.0 -> lower=-0.00000000000000033307 upper=2.00290417450818303280 effort=1.0 velocity=1.0
- joint _ring_link_j01: limit lower=-0.00000000000000027756 upper=2.15805382455002581210 effort=10.0 velocity=1.0 -> lower=-0.00000000000000027756 upper=2.15805382455002581210 effort=1.0 velocity=1.0
- joint _ring_proximal_j01: limit lower=-0.00000000000000022204 upper=2.42566926019509709889 effort=10.0 velocity=1.0 -> lower=-0.00000000000000022204 upper=2.42566926019509709889 effort=1.0 velocity=1.0
- joint _thumb_chassis_j01: limit lower=0.00000002107342389479 upper=1.53339620392031616980 effort=10.0 velocity=1.0 -> lower=0.00000002107342389479 upper=1.53339620392031616980 effort=1.0 velocity=1.0
- joint _thumb_distal_j01: limit lower=-0.00000000000000033307 upper=1.70697629504807113499 effort=10.0 velocity=1.0 -> lower=-0.00000000000000033307 upper=1.70697629504807113499 effort=1.0 velocity=1.0
- joint _thumb_follower_j01: limit lower=-0.00000000000000022204 upper=1.49972422122050308424 effort=10.0 velocity=1.0 -> lower=-0.00000000000000022204 upper=1.49972422122050308424 effort=1.0 velocity=1.0
- joint _thumb_link_j01: limit lower=-0.00000000000000016653 upper=1.22879127474338734061 effort=10.0 velocity=1.0 -> lower=-0.00000000000000016653 upper=1.22879127474338734061 effort=1.0 velocity=1.0
- joint _thumb_proximal_j01: limit lower=-0.00000000000000016653 upper=1.15235501787369631899 effort=10.0 velocity=1.0 -> lower=-0.00000000000000016653 upper=1.15235501787369631899 effort=1.0 velocity=1.0
