Commit message: adição de braço robótico

File: install/hand_pack/share/hand_pack/urdf/hand.xacro (robot description, xacro)
@@ -1,14 +1,20 @@
 <?xml version="1.0"?>
 <robot xmlns:xacro="http://www.ros.org/wiki/xacro" name="hj_hand">
-    <link name="base_link">
-        <visual>
-            <geometry>
-                <box size="0.01 0.10 0.01"/> <!-- Ajuste conforme necessário -->
-            </geometry>
-            <material name="white">
-                <color rgba="1 1 1 1"/>
-            </material>
-        </visual>
-    </link>
+  <!-- Definição da base da mão -->
+    <xacro:macro name="base_link" params="parent">
+        <link name="hand_base_link">
+            <visual>
+                <geometry>
+                    <mesh filename="package://hand_pack/urdf/mesh/hand_model.stl"/>
+                </geometry>
+            </visual>
+        </link>
+        <!-- Junta a mão ao braço -->
+        <joint name="hand_mount" type="fixed">
+            <parent link="${parent}"/>
+            <child link="hand_base_link"/>
+            <origin xyz="0 0 0.05" rpy="0 0 0"/>
+        </joint>
+    </xacro:macro>
       <xacro:macro name="hj_hand" params="parent *origin">
             <xacro:include filename="$(find hand_pack)/urdf/hj_hand_transmission.xacro" />
@@ -31,5 +37,5 @@
             <xacro:property name="motor_max_upper" value="0.0103" /> <!--joint origin-->
 <!--****************WRIST PLATE************************* -->
-      <link name="wrist_plate">
+      <link name="hand_wrist_plate">
             <visual>
                   <geometry>
@@ -48,8 +54,8 @@
             </collision>
       </link>
-      <joint name="wrist_plate_joint" type="fixed">
+      <joint name="hand_wrist_plate_joint" type="fixed">
             <origin xyz="0 0 0" rpy="0 0 0"/>
             <parent link="${parent}"/>
-            <child link="wrist_plate"/>
+            <child link="hand_wrist_plate"/>
             <limit lower="0.0" upper="0.0" effort="0.0" velocity="0.0"/>
       </joint>
@@ -84,6 +90,6 @@
             </inertial>
       </link>
-      <joint name="hand_wrist_plate_to_hand_palm" type="fixed">
-            <parent link="wrist_plate"/>
+      <joint name="hand_hand_wrist_plate_to_hand_palm" type="fixed">
+            <parent link="hand_wrist_plate"/>
             <child link="hand_palm"/>
             <origin xyz="0 0 .026"/>
@@ -1222,6 +1228,3 @@
       <!--motor little  end-->
 </xacro:macro>
-<xacro:hj_hand parent="base_link">
-    <origin xyz="0 0 0" rpy="0 0 0"/>
-</xacro:hj_hand>
 </robot>
