Commit message: mega simull no webots -ajeitar as bounding box

File: install/hand_pack/share/hand_pack/urdf/hand.xacro (robot description, xacro)
@@ -1,1227 +1 @@
-<?xml version="1.0"?>
-<robot xmlns:xacro="http://www.ros.org/wiki/xacro" name="hj_hand">
-    <link name="base_link">
-        <visual>
-            <geometry>
-                <box size="0.001 0.001 0.001"/>
-            </geometry>
-            <material name="white">
-                <color rgba="1 1 1 1"/>
-            </material>
-        </visual>
-    </link>
-      <xacro:macro name="hj_hand" params="parent *origin">
-            <xacro:include filename="$(find hand_pack)/urdf/hj_hand_transmission.xacro" />
-            <xacro:include filename="$(find hand_pack)/urdf/hj_hand_gazebo.xacro" />
-            <xacro:property name="motor_x" value="0.016" />
-            <xacro:property name="motor_y" value="0.035" />
-            <xacro:property name="motor_z" value="0.02" />
-            <xacro:property name="pris_x" value="0.005" />
-            <xacro:property name="pris_y" value="0.005" />
-            <xacro:property name="pris_z" value="0.025" />
-            <xacro:property name="knucle_mass" value="0.010" />
-            <xacro:property name="MCP_mass" value="0.0125" />
-            <xacro:property name="PIP_mass" value="0.0125" />
-            <xacro:property name="DIP_mass" value="0.0025" />
-            <xacro:property name="motor_mass" value="0.015" />
-            <xacro:property name="motor_joint_x" value="0.0" />
-            <xacro:property name="motor_joint_y" value="-0.0145" />
-            <xacro:property name="motor_joint_z" value="0.006" />
-            <xacro:property name="eef_offset_z" value="0.025725" />
-            <xacro:property name="motor_max_upper" value="0.0103" /> <!--joint origin-->
-<!--****************WRIST PLATE************************* -->
-      <link name="wrist_plate">
-            <visual>
-                  <geometry>
-                        <mesh filename="package://hand_pack/urdf/mesh/F03_AL_link_hand_wrist_part.stl" scale="0.001 0.001 0.001"/>
-                  </geometry>
-                  <origin xyz = "0.0 0.0 0.0" rpy = "1.57 0.0 0.0"/>
-                  <material name="white">
-                        <color rgba="0.85 0.85 0.85 1"/>
-                  </material>
-            </visual>
-            <collision>
-                  <geometry>
-                        <mesh filename="package://hand_pack/urdf/mesh/F03_AL_link_hand_wrist_part.stl" scale="0.001 0.001 0.001"/>
-                  </geometry>
-                  <origin xyz = "0.0 0.0 0.0" rpy = "1.57 0.0 0.0"/>
-            </collision>
-      </link>
-      <joint name="wrist_plate_joint" type="fixed">
-            <origin xyz="0 0 0" rpy="0 0 0"/>
-            <parent link="${parent}"/>
-            <child link="wrist_plate"/>
-            <limit lower="0.0" upper="0.0" effort="0.0" velocity="0.0"/>
-      </joint>
-      <!--**************** hand palm*************************-->
-      <xacro:property name="hand_palm_x" value="0.0" />
-      <xacro:property name="hand_palm_y" value="0.0162" />
-      <xacro:property name="hand_palm_z" value="0.030" />
-      <xacro:property name="hand_palm_r" value="3.14" />
-      <xacro:property name="hand_palm_p" value="4.71" />
-      <xacro:property name="hand_palm_yaw" value="0.0" />
-      <link name="hand_palm">
-            <visual>
-                  <geometry>
-                  <mesh filename="package://hand_pack/urdf/mesh/F03_AL_palm.stl" scale="0.001 0.001 0.001"/>
-                  </geometry>
-                  <origin xyz = "${hand_palm_x} ${hand_palm_y} ${hand_palm_z}" rpy = "${hand_palm_r} ${hand_palm_p} ${hand_palm_yaw}"/>
-                  <material name="lightgrey">
-                  <color rgba="0.5 0.5 0.5 1.0"/>
-                  </material>
-            </visual>
-            <collision>
-                  <geometry>
-                  <mesh filename="package://hand_pack/urdf/mesh/F03_AL_palm.stl" scale="0.001 0.001 0.001"/>
-                  </geometry>
-                  <origin xyz = "${hand_palm_x} ${hand_palm_y} ${hand_palm_z}" rpy = "${hand_palm_r} ${hand_palm_p} ${hand_palm_yaw}"/>
-            </collision>
-            <inertial>
-                  <mass value="0.09"/>
-                  <inertia ixx="1.0e-03" ixy="0.0" ixz="0.0"
-               iyy="1.0e-03" iyz="0.0"
-               izz="1.0e-03" />
-            </inertial>
-      </link>
-      <joint name="hand_wrist_plate_to_hand_palm" type="fixed">
-            <parent link="wrist_plate"/>
-            <child link="hand_palm"/>
-            <origin xyz="0 0 .026"/>
-      </joint>
-      <!--****************4 fingers*************************-->
-      <xacro:property name="knuckle_4finger_x" value="-0.0313" /> <!--joint origin-->
-      <xacro:property name="knuckle_4finger_y" value="0.0160" />
-      <xacro:property name="knuckle_4finger_z" value="0.0295" />
-      <xacro:property name="knuckle_roll" value="0.0" />        <!--link orientation -->
-      <xacro:property name="knuckle_pitch" value="-1.57" />
-      <xacro:property name="knuckle_yaw" value="-3.14" />
-      <link name="knuckle_index">
-      <visual>
-            <geometry>
-            <mesh filename="package://hand_pack/urdf/mesh/F03_Finger_base.stl" scale="0.001 0.001 0.001"/>
-            </geometry>
-            <origin xyz = "0.0 0.0 0.0" rpy = "${knuckle_roll} ${knuckle_pitch} ${knuckle_yaw}"/>
-            <material name="white">
-            </material>
-      </visual>
-      <collision>
-            <geometry>
-            <mesh filename="package://hand_pack/urdf/mesh/F03_Finger_base.stl" scale="0.001 0.001 0.001"/>
-            </geometry>
-            <origin xyz = "0.0 0.0 0.0" rpy = "${knuckle_roll} ${knuckle_pitch} ${knuckle_yaw}"/>
-      </collision>
-      <inertial>
-            <mass value="${knucle_mass}"/>
-            <inertia ixx="1.0e-03" ixy="0.0" ixz="0.0"
-               iyy="1.0e-03" iyz="0.0"
-               izz="1.0e-03" />
-      </inertial>
-      </link>
-      <joint name="knuckle_index_joint" type="fixed">
-      <parent link="hand_palm"/>
-      <child link="knuckle_index"/>
-      <origin xyz ="${knuckle_4finger_x}
-                        ${knuckle_4finger_y}
-                        ${knuckle_4finger_z}"/>
-      </joint>
-      <link name="knuckle_middle">
-      <visual>
-            <geometry>
-            <mesh filename="package://hand_pack/urdf/mesh/F03_Finger_base.stl" scale="0.001 0.001 0.001"/>
-            </geometry>
-            <origin xyz = "0.0 0.0 0.0" rpy = "${knuckle_roll} ${knuckle_pitch} ${knuckle_yaw}"/>
-            <material name="white">
-            </material>
-      </visual>
-      <collision>
-            <geometry>
-            <mesh filename="package://hand_pack/urdf/mesh/F03_Finger_base.stl" scale="0.001 0.001 0.001"/>
-            </geometry>
-            <origin xyz = "0.0 0.0 0.0" rpy = "${knuckle_roll} ${knuckle_pitch} ${knuckle_yaw}"/>
-      </collision>
-      <inertial>
-            <mass value="${knucle_mass}"/>
-            <inertia ixx="1.0e-03" ixy="0.0" ixz="0.0"
-               iyy="1.0e-03" iyz="0.0"
-               izz="1.0e-03" />
-      </inertial>
-      </link>
-            <joint name="knuckle_middle_joint" type="fixed">
-            <parent link="hand_palm"/>
-            <child link="knuckle_middle"/>
-            <origin xyz ="${knuckle_4finger_x + 0.0210}
-                              ${knuckle_4finger_y}
-                              ${knuckle_4finger_z}"/>
-      </joint>
-      <link name="knuckle_ring">
-            <visual>
-                  <geometry>
-                  <mesh filename="package://hand_pack/urdf/mesh/F03_Finger_base.stl" scale="0.001 0.001 0.001"/>
-                  </geometry>
-                  <origin xyz = "0.0 0.0 0.0" rpy = "${knuckle_roll} ${knuckle_pitch} ${knuckle_yaw}"/>
-                  <material name="white">
-                  </material>
-            </visual>
-            <collision>
-                  <geometry>
-                  <mesh filename="package://hand_pack/urdf/mesh/F03_Finger_base.stl" scale="0.001 0.001 0.001"/>
-                  </geometry>
-                  <origin xyz = "0.0 0.0 0.0" rpy = "${knuckle_roll} ${knuckle_pitch} ${knuckle_yaw}"/>
-            </collision>
-            <inertial>
-                  <mass value="${knucle_mass}"/>
-                  <inertia ixx="1.0e-03" ixy="0.0" ixz="0.0"
-               iyy="1.0e-03" iyz="0.0"
-               izz="1.0e-03" />
-            </inertial>
-      </link>
-            <joint name="knuckle_ring_joint" type="fixed">
-                  <parent link="hand_palm"/>
-                  <child link="knuckle_ring"/>
-                  <origin xyz ="${knuckle_4finger_x + 0.0420}
-                                    ${knuckle_4finger_y}
-                                    ${knuckle_4finger_z}"/>
-            </joint>
-      <link name="knuckle_little">
-            <visual>
-                  <geometry>
-                  <mesh filename="package://hand_pack/urdf/mesh/F03_Finger_base.stl" scale="0.001 0.001 0.001"/>
-                  </geometry>
-                  <origin xyz = "0.0 0.0 0.0" rpy = "${knuckle_roll} ${knuckle_pitch} ${knuckle_yaw}"/>
-                  <material name="white">
-                  </material>
-            </visual>
-            <collision>
-                  <geometry>
-                  <mesh filename="package://hand_pack/urdf/mesh/F03_Finger_base.stl" scale="0.001 0.001 0.001"/>
-                  </geometry>
-                  <origin xyz = "0.0 0.0 0.0" rpy = "${knuckle_roll} ${knuckle_pitch} ${knuckle_yaw}"/>
-            </collision>
-            <inertial>
-                  <mass value="${knucle_mass}"/>
-                  <inertia ixx="1.0e-03" ixy="0.0" ixz="0.0"
-               iyy="1.0e-03" iyz="0.0"
-               izz="1.0e-03" />
-            </inertial>
-      </link>
-      <joint name="knuckle_little_joint" type="fixed">
-            <parent link="hand_palm"/>
-            <child link="knuckle_little"/>
-            <origin xyz ="${knuckle_4finger_x + 0.0630}
-                              ${knuckle_4finger_y}
-                              ${knuckle_4finger_z}"/>
-      </joint>
-      <!--****************Thumb part*************************-->
-      <xacro:property name="knuckle_thumb_x" value="0.0345" /> <!--joint origin-->
-      <xacro:property name="knuckle_thumb_y" value="0.0162" />
-      <xacro:property name="knuckle_thumb_z" value="0.0186" />
-      <xacro:property name="thumb_joint_joint_x" value="-0.0558" /> <!--joint origin-->
-      <xacro:property name="thumb_joint_joint_y" value="-0.00675" />
-      <xacro:property name="thumb_joint_joint_z" value="-0.0" />
-      <xacro:property name="thumb_x" value="0.00" /> <!--link offset-->
-      <xacro:property name="thumb_y" value="0" />
-      <xacro:property name="thumb_z" value="-0.005" />
-      <xacro:property name="thumb_roll" value="0.0" /> <!--joint offset-->
-      <xacro:property name="thumb_pitch" value="0" />
-      <xacro:property name="thumb_yaw" value="3.14" />
-      <xacro:property name="thumb_link_MCP_x" value="0.00955" /> <!--link offset-->
-      <xacro:property name="thumb_link_MCP_y" value="0.0" />
-      <xacro:property name="thumb_link_MCP_z" value="0.00415" />
-      <xacro:property name="thumb_link_DIP_x" value="0.00255" /> <!--link offset-->
-      <xacro:property name="thumb_link_DIP_y" value="0.00" />
-      <xacro:property name="thumb_link_DIP_z" value="0.00726" />
-      <xacro:property name="thumb_finger_roll" value="-1.57" /> <!--link offset-->
-      <xacro:property name="thumb_finger_pitch" value="0" />
-      <xacro:property name="thumb_finger_yaw" value="3.14" />
-      <xacro:property name="thumb_joint_MCP_x" value="-0.031" /> <!--joint origin-->
-      <xacro:property name="thumb_joint_MCP_y" value="-0.0055" />
-      <xacro:property name="thumb_joint_MCP_z" value="-0.000" />
-      <xacro:property name="thumb_joint_DIP_x" value="-0.0298" /> <!--joint origin-->
-      <xacro:property name="thumb_joint_DIP_y" value="-0.00" />
-      <xacro:property name="thumb_joint_DIP_z" value="-0.0042" />
-      <link name="knuckle_thumb">
-            <visual>
-                  <geometry>
-                  <mesh filename="package://hand_pack/urdf/mesh/F03_Thumb_base.stl" scale="0.001 0.001 0.001"/>
-                  </geometry>
-                  <origin xyz = "0.0 0.0 0.0" rpy = "${knuckle_roll} 0.0 ${knuckle_yaw}"/>
-                  <material name="white">
-                  </material>
-            </visual>
-            <collision>
-                  <geometry>
-                  <mesh filename="package://hand_pack/urdf/mesh/F03_Thumb_base.stl" scale="0.001 0.001 0.001"/>
-                  </geometry>
-                  <origin xyz = "0.0 0.0 0.0" rpy = "${knuckle_roll} 0.0 ${knuckle_yaw}"/>
-            </collision>
-            <inertial>
-                  <mass value="${knucle_mass}"/>
-                  <inertia ixx="1.0e-03" ixy="0.0" ixz="0.0"
-               iyy="1.0e-03" iyz="0.0"
-               izz="1.0e-03" />
-            </inertial>
-      </link>
-      <joint name="knuckle_thumb_joint" type="fixed">
-            <parent link="hand_palm"/>
-            <child link="knuckle_thumb"/>
-            <origin xyz = "${knuckle_thumb_x}
-                           ${knuckle_thumb_y}
-                           ${knuckle_thumb_z}"/>
-      </joint>
-      <!-- Thumb finger -->
-      <link name="thumb_joint">
-      <visual>
-            <geometry>
-                  <mesh filename="package://hand_pack/urdf/mesh/F03_Thumb_joint.stl" scale="0.001 0.001 0.001"/>
-            </geometry>
-                  <origin xyz = "${thumb_x} ${thumb_y} ${thumb_z}" rpy = "${thumb_roll} ${thumb_pitch} ${thumb_yaw}"/>
-            <material name="white">
-            </material>
-      </visual>
-      <collision>
-            <geometry>
-                  <mesh filename="package://hand_pack/urdf/mesh/F03_Thumb_joint.stl" scale="0.001 0.001 0.001"/>
-            </geometry>
-            <origin xyz = "${thumb_x} ${thumb_y} ${thumb_z}" rpy = "${thumb_roll} ${thumb_pitch} ${thumb_yaw}"/>
-      </collision>
-      <inertial>
-            <mass value="${motor_mass}"/>
-            <inertia ixx="1.0e-03" ixy="0.0" ixz="0.0"
-               iyy="1.0e-03" iyz="0.0"
-               izz="1.0e-03" />
-      </inertial>
-      </link>
-      <joint name="thumb_jo_joint" type="revolute">
-            <axis xyz="0 0 -1"/>    <!--z axis rotate -->
-            <limit effort="1000.0" lower="0.0" upper="1.8" velocity="0.5"/>
-            <parent link="knuckle_thumb"/>
-            <child link="thumb_joint"/>
-            <origin xyz="${thumb_joint_joint_x}
-                         ${thumb_joint_joint_y}
-                         ${thumb_joint_joint_z}" rpy = "0.0 0.0 -0.6021" />
-            <joint_properties damping="1.0" friction="0.0"/>
-            <mimic joint="pris_thumb_jo_joint" multiplier="100.00" offset="0.0" />
-      </joint>
-      <link name="thumb_MCP">
-      <visual>
-            <geometry>
-                  <mesh filename="package://hand_pack/urdf/mesh/F03_AL_link_MCP.stl" scale="0.001 0.001 0.001"/>
-            </geometry>
-                  <origin xyz = "${thumb_link_MCP_x} ${thumb_link_MCP_y} ${thumb_link_MCP_z}"
-                          rpy = "${thumb_finger_roll} ${thumb_finger_pitch} ${thumb_finger_yaw}"/>
-            <material name="white">
-            </material>
-      </visual>
-      <collision>
-            <geometry>
-            <mesh filename="package://hand_pack/urdf/mesh/F03_AL_link_MCP.stl" scale="0.001 0.001 0.001"/>
-            </geometry>
-            <origin xyz = "${thumb_link_MCP_x} ${thumb_link_MCP_y} ${thumb_link_MCP_z}" rpy = "${thumb_finger_roll} ${thumb_finger_pitch} ${thumb_finger_yaw}"/>
-      </collision>
-      <inertial>
-            <mass value="${MCP_mass}"/>
-            <inertia ixx="1.0e-03" ixy="0.0" ixz="0.0"
-               iyy="1.0e-03" iyz="0.0"
-               izz="1.0e-03" />
-      </inertial>
-      </link>
-      <joint name="thumb_MCP_joint" type="revolute">
-            <axis xyz="0 1 0"/>
-            <limit effort="1000.0" lower="0.0" upper="1.0" velocity="0.5"/>
-            <parent link="thumb_joint"/>
-            <child link="thumb_MCP"/>
-            <origin xyz="${thumb_joint_MCP_x}
-                         ${thumb_joint_MCP_y}
-                         ${thumb_joint_MCP_z}" rpy = "0.0 0.4538 0.0"/>
-            <joint_properties damping="1.0" friction="0.0"/>
-            <mimic joint="pris_thumb_DIP_joint" multiplier="100.00" offset="0.0" />
-      </joint>
-      <link name="thumb_DIP">
-      <visual>
-            <geometry>
-                  <mesh filename="package://hand_pack/urdf/mesh/F03_AL_link_DIP.stl" scale="0.001 0.001 0.001"/>
-            </geometry>
-                  <origin xyz = "${thumb_link_DIP_x} ${thumb_link_DIP_y} ${thumb_link_DIP_z}" rpy = "${thumb_finger_roll} ${thumb_finger_pitch} ${thumb_finger_yaw}"/>
-            <material name="lightyellow">
-            <color rgba="1.0 1.0 0.3 1.0"/>
-            </material>
-      </visual>
-      <collision>
-            <geometry>
-            <mesh filename="package://hand_pack/urdf/mesh/F03_AL_link_DIP.stl" scale="0.001 0.001 0.001"/>
-            </geometry>
-            <origin xyz = "${thumb_link_DIP_x} ${thumb_link_DIP_y} ${thumb_link_DIP_z}" rpy = "${thumb_finger_roll} ${thumb_finger_pitch} ${thumb_finger_yaw}"/>
-      </collision>
-      <inertial>
-            <mass value="${DIP_mass}"/>
-            <inertia ixx="1.0e-03" ixy="0.0" ixz="0.0"
-               iyy="1.0e-03" iyz="0.0"
-               izz="1.0e-03" />
-      </inertial>
-      </link>
-      <joint name="thumb_DIP_joint" type="revolute">
-            <axis xyz="0 1 0"/>
-            <limit effort="1000.0" lower="0.0" upper="0.8" velocity="0.5"/>
-            <parent link="thumb_MCP"/>
-            <child link="thumb_DIP"/>
-            <origin xyz="${thumb_joint_DIP_x}
-                         ${thumb_joint_DIP_y}
-                         ${thumb_joint_DIP_z}" rpy = "0.0 0.0 0.0"/>
-            <joint_properties damping="1.0" friction="0.0"/>
-            <mimic joint="pris_thumb_DIP_joint" multiplier="100.00" offset="0.0" />
-      </joint>
-      <link name="ee_thumb_link">
-            <collision>
-                  <geometry>
-                        <box size="0.0001 0.0001 0.0001"/>
-                  </geometry>
-                  <origin xyz="0.0 0.0 0.0" rpy="0.0 0.0 0.0"/>
-            </collision>
-      </link>
-      <joint name="ee_th_joint" type="fixed">
-            <parent link="thumb_DIP"/>
-            <child link="ee_thumb_link"/>
-            <origin xyz="${-eef_offset_z} 0.0 0.0 " rpy="0.0 0.0 0.0"/>
-      </joint>
-      <!-- Thumb finger end -->
-      <!-- Thumb motor -->
-      <xacro:property name="motor_th_joint_x" value="-0.008" />  <!-- joint offset -->
-      <xacro:property name="motor_th_joint_y" value="-0.015" />
-      <xacro:property name="motor_th_joint_z" value="-0.000" />
-      <xacro:property name="motor_dip_joint_x" value="0.0125" />  <!-- joint offset -->
-      <xacro:property name="motor_dip_joint_y" value="-0.0055" />
-      <xacro:property name="motor_dip_joint_z" value="-0.015" />
-      <link name="motor_thumb_jo">
-            <visual>
-                  <geometry>
-                  <box size="${motor_x} ${motor_y} ${motor_z}"/>
-                  </geometry>
-                  <origin xyz="0 .02 0"/>
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
File: install/hand_pack/share/hand_pack/urdf/hj_hand_gazebo.xacro (robot description, xacro)
@@ -1,73 +1 @@
-<?xml version="1.0"?>
-<robot xmlns:xacro="http://ros.org/wiki/xacro">
-    <gazebo reference="pris_thumb_jo">
-      <selfCollide>true</selfCollide>
-    </gazebo>
-    <gazebo reference="pris_thumb_DIP">
-      <selfCollide>true</selfCollide>
-    </gazebo>
-    <gazebo reference="pris_index">
-      <selfCollide>true</selfCollide>
-    </gazebo>
-    <gazebo reference="pris_middle">
-      <selfCollide>true</selfCollide>
-    </gazebo>
-    <gazebo reference="pris_ring">
-      <selfCollide>true</selfCollide>
-    </gazebo>
-    <gazebo reference="pris_little">
-      <selfCollide>true</selfCollide>
-    </gazebo>
-<!-- fingers-->
-    <gazebo reference="thumb_joint">
-      <selfCollide>true</selfCollide>
-    </gazebo>
-    <gazebo reference="thumb_MCP">
-      <selfCollide>true</selfCollide>
-    </gazebo>
-    <gazebo reference="thumb_DIP">
-      <selfCollide>true</selfCollide>
-    </gazebo>
-    <gazebo reference="index_MCP">
-      <selfCollide>true</selfCollide>
-    </gazebo>
-    <gazebo reference="index_PIP">
-      <selfCollide>true</selfCollide>
-    </gazebo>
-    <gazebo reference="index_DIP">
-      <selfCollide>true</selfCollide>
-    </gazebo>
-    <gazebo reference="middle_MCP">
-      <selfCollide>true</selfCollide>
-    </gazebo>
-    <gazebo reference="middle_PIP">
-      <selfCollide>true</selfCollide>
-    </gazebo>
-    <gazebo reference="middle_DIP">
-      <selfCollide>true</selfCollide>
-    </gazebo>
-    <gazebo reference="ring_MCP">
-      <selfCollide>true</selfCollide>
-    </gazebo>
-    <gazebo reference="ring_PIP">
-      <selfCollide>true</selfCollide>
-    </gazebo>
-    <gazebo reference="ring_DIP">
-      <selfCollide>true</selfCollide>
-    </gazebo>
-    <gazebo reference="little_MCP">
-      <selfCollide>true</selfCollide>
-    </gazebo>
-    <gazebo reference="little_PIP">
-      <selfCollide>true</selfCollide>
-    </gazebo>
-    <gazebo reference="little_DIP">
-      <selfCollide>true</selfCollide>
-    </gazebo>
-    <gazebo>
-      <plugin name="gazebo_ros_control" filename="libgazebo_ros_control.so">
-        <robotNamespace>/hj_hand_chain</robotNamespace>
-        <robotSimType>gazebo_ros_control/DefaultRobotHWSim</robotSimType>
-      </plugin>
-    </gazebo>
-</robot>
+/home/lucas-pc/RoboticArm/build/hand_pack/urdf/hj_hand_gazebo.xacro
