Commit message: controladores da mão

File: install/hand_pack/share/hand_pack/urdf/linear_covvi_hand_right_scaled.urdf (robot description, URDF)
Before this commit: robot covvi_hand_right, 87 links, 86 joints
Links:
- link Index_driver_link: mass 1 -> 0
- link Little_driver_link: mass 1 -> 0
- link Middle_driver_link: mass 1 -> 0
- link Ring_driver_link: mass 1 -> 0
- link Rotate_driver_link: mass 1 -> 0
- link Thumb_driver_link: mass 1 -> 0
- link __base_link: mass 1 -> 0
- link _base_link: mass 1 -> 0
- link _index_distal_l1: mass 1 -> 0
- link _index_follower_l1: mass 1 -> 0
- link _index_knuckle_l1: mass 1 -> 0
- link _index_link_l1: mass 1 -> 0
- link _index_proximal_l1: mass 1 -> 0
- link _lisa_l1: mass 1 -> 0
- link _little_distal_l1: mass 1 -> 0
- link _little_follower_l1: mass 1 -> 0
- link _little_knuckle_l1: mass 1 -> 0
- link _little_link_l1: mass 1 -> 0
- link _little_proximal_l1: mass 1 -> 0
- link _middle_distal_l1: mass 1 -> 0
- link _middle_follower_l1: mass 1 -> 0
- link _middle_knuckle_l1: mass 1 -> 0
- link _middle_link_l1: mass 1 -> 0
- link _middle_proximal_l1: mass 1 -> 0
- link _ring_distal_l1: mass 1 -> 0
- link _ring_follower_l1: mass 1 -> 0
- link _ring_knuckle_l1: mass 1 -> 0
- link _ring_link_l1: mass 1 -> 0
- link _ring_proximal_l1: mass 1 -> 0
- link _thumb_chassis_l1: mass 1 -> 0
- link _thumb_distal_l1: mass 1 -> 0
- link _thumb_follower_l1: mass 1 -> 0
- link _thumb_link_l1: mass 1 -> 0
- link _thumb_proximal_l1: mass 1 -> 0
- link base_link: geometry visual mesh filename=package://hand_pack/urdf/linear_meshes/right_base_link.STL scale=0.00125 0.00125 0.00125
- link index_distal: geometry visual mesh filename=package://hand_pack/urdf/linear_meshes/right_index_distal.S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 scale=0.00125 0.00125 0.00125
- link index_follower: geometry visual mesh filename=package://hand_pack/urdf/linear_meshes/right_index_follower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 scale=0.00125 0.00125 0.00125
- link index_knuckle: geometry visual mesh filename=package://hand_pack/urdf/linear_meshes/right_index_knuckle.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 scale=0.00125 0.00125 0.00125
- link index_link: geometry visual mesh filename=package://hand_pack/urdf/linear_meshes/right_index_link.STL scale=0.00125 0.00125 0.00125
- link index_proximal: geometry visual mesh filename=package://hand_pack/urdf/linear_meshes/right_index_proximal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 scale=0.00125 0.00125 0.00125
- link lisa: geometry visual mesh filename=package://hand_pack/urdf/linear_meshes/right_lisa.STL scale=0.00125 0.00125 0.00125
- link little_distal: geometry visual mesh filename=package://hand_pack/urdf/linear_meshes/right_little_distal.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 scale=0.00125 0.00125 0.00125
- link little_follower: geometry visual mesh filename=package://hand_pack/urdf/linear_meshes/right_little_followe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 scale=0.00125 0.00125 0.00125
- link little_knuckle: geometry visual mesh filename=package://hand_pack/urdf/linear_meshes/right_little_knuckle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 scale=0.00125 0.00125 0.00125
- link little_link: geometry visual mesh filename=package://hand_pack/urdf/linear_meshes/right_little_link.STL scale=0.00125 0.00125 0.00125
- link little_proximal: geometry visual mesh filename=package://hand_pack/urdf/linear_meshes/right_little_proxima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 scale=0.00125 0.00125 0.00125
- link middle_distal: geometry visual mesh filename=package://hand_pack/urdf/linear_meshes/right_middle_distal.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 scale=0.00125 0.00125 0.00125
- link middle_follower: geometry visual mesh filename=package://hand_pack/urdf/linear_meshes/right_middle_followe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 scale=0.00125 0.00125 0.00125
- link middle_knuckle: geometry visual mesh filename=package://hand_pack/urdf/linear_meshes/right_middle_knuckle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 scale=0.00125 0.00125 0.00125
- link middle_link: geometry visual mesh filename=package://hand_pack/urdf/linear_meshes/right_middle_link.STL scale=0.00125 0.00125 0.00125
- link middle_proximal: geometry visual mesh filename=package://hand_pack/urdf/linear_meshes/right_middle_proxima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 scale=0.00125 0.00125 0.00125
- link ring_distal: geometry visual mesh filename=package://hand_pack/urdf/linear_meshes/right_ring_distal.STL scale=0.00125 0.00125 0.00125
- link ring_follower: geometry visual mesh filename=package://hand_pack/urdf/linear_meshes/right_ring_follower.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 scale=0.00125 0.00125 0.00125
- link ring_knuckle: geometry visual mesh filename=package://hand_pack/urdf/linear_meshes/right_ring_knuckle.S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 scale=0.00125 0.00125 0.00125
- link ring_link: geometry visual mesh filename=package://hand_pack/urdf/linear_meshes/right_ring_link.STL scale=0.00125 0.00125 0.00125
- link ring_proximal: geometry visual mesh filename=package://hand_pack/urdf/linear_meshes/right_ring_proximal.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 scale=0.00125 0.00125 0.00125
- link thumb_chassis: geometry visual mesh filename=package://hand_pack/urdf/linear_meshes/right_thumb_chassis.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 scale=0.00125 0.00125 0.00125
- link thumb_distal: geometry visual mesh filename=package://hand_pack/urdf/linear_meshes/right_thumb_distal.S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 scale=0.00125 0.00125 0.00125
- link thumb_follower: geometry visual mesh filename=package://hand_pack/urdf/linear_meshes/right_thumb_follower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 scale=0.00125 0.00125 0.00125
- link thumb_link: geometry visual mesh filename=package://hand_pack/urdf/linear_meshes/right_thumb_link.STL scale=0.00125 0.00125 0.00125
- link thumb_proximal: geometry visual mesh filename=package://hand_pack/urdf/linear_meshes/right_thumb_proximal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 scale=0.00125 0.00125 0.00125
