Commit message: simulação boa no gazebo

File: src/hand_pack/urdf/linear_covvi_hand_gazebo.urdf (robot description, URDF)
Before this commit: robot covvi_hand_right, 88 links, 87 joints
Links:
- removed link __base_link
- removed link _base_link
- added link base_footprint
- link Index_driver_link: mass 0.005 -> 1
- link Little_driver_link: mass 0.005 -> 1
- link Middle_driver_link: mass 0.005 -> 1
- link Ring_driver_link: mass 0.005 -> 1
- link Rotate_driver_link: mass 0.005 -> 1
- link Thumb_driver_link: mass 0.005 -> 1
- link _index_distal_l0: mass 0.03 -> 0.01; geometry visual box size=0 0 0
- link _index_distal_l1: mass 0.02 -> 1; geometry visual box size=0 0 0
- link _index_follower_l0: mass 0.03 -> 0.01; geometry visual box size=0 0 0
- link _index_follower_l1: mass 0.02 -> 1; geometry visual box size=0 0 0
- link _index_knuckle_l0: mass 0.03 -> 0.01; geometry visual box size=0 0 0
- link _index_knuckle_l1: mass 0.02 -> 1; geometry visual box size=0 0 0
- link _index_link_l0: mass 0.03 -> 0.01; geometry visual box size=0 0 0
- link _index_link_l1: mass 0.02 -> 1; geometry visual box size=0 0 0
- link _index_proximal_l0: mass 0.03 -> 0.01; geometry visual box size=0 0 0
- link _index_proximal_l1: mass 0.02 -> 1; geometry visual box size=0 0 0
- link _lisa_l0: mass 0.005 -> 0.01; geometry visual box size=0 0 0
- link _lisa_l1: mass 0.005 -> 1; geometry visual box size=0 0 0
- link _little_distal_l0: mass 0.03 -> 0.01; geometry visual box size=0 0 0
- link _little_distal_l1: mass 0.02 -> 1; geometry visual box size=0 0 0
- link _little_follower_l0: mass 0.03 -> 0.01; geometry visual box size=0 0 0
- link _little_follower_l1: mass 0.02 -> 1; geometry visual box size=0 0 0
- link _little_knuckle_l0: mass 0.03 -> 0.01; geometry visual box size=0 0 0
- link _little_knuckle_l1: mass 0.02 -> 1; geometry visual box size=0 0 0
- link _little_link_l0: mass 0.03 -> 0.01; geometry visual box size=0 0 0
- link _little_link_l1: mass 0.02 -> 1; geometry visual box size=0 0 0
- link _little_proximal_l0: mass 0.03 -> 0.01; geometry visual box size=0 0 0
- link _little_proximal_l1: mass 0.02 -> 1; geometry visual box size=0 0 0
- link _middle_distal_l0: mass 0.03 -> 0.01; geometry visual box size=0 0 0
- link _middle_distal_l1: mass 0.02 -> 1; geometry visual box size=0 0 0
- link _middle_follower_l0: mass 0.03 -> 0.01; geometry visual box size=0 0 0
- link _middle_follower_l1: mass 0.02 -> 1; geometry visual box size=0 0 0
- link _middle_knuckle_l0: mass 0.03 -> 0.01; geometry visual box size=0 0 0
- link _middle_knuckle_l1: mass 0.02 -> 1; geometry visual box size=0 0 0
- link _middle_link_l0: mass 0.03 -> 0.01; geometry visual box size=0 0 0
- link _middle_link_l1: mass 0.02 -> 1; geometry visual box size=0 0 0
- link _middle_proximal_l0: mass 0.03 -> 0.01; geometry visual box size=0 0 0
- link _middle_proximal_l1: mass 0.02 -> 1; geometry visual box size=0 0 0
- link _ring_distal_l0: mass 0.03 -> 0.01; geometry visual box size=0 0 0
- link _ring_distal_l1: mass 0.02 -> 1; geometry visual box size=0 0 0
- link _ring_follower_l0: mass 0.03 -> 0.01; geometry visual box size=0 0 0
- link _ring_follower_l1: mass 0.02 -> 1; geometry visual box size=0 0 0
- link _ring_knuckle_l0: mass 0.03 -> 0.01; geometry visual box size=0 0 0
- link _ring_knuckle_l1: mass 0.02 -> 1; geometry visual box size=0 0 0
- link _ring_link_l0: mass 0.03 -> 0.01; geometry visual box size=0 0 0
- link _ring_link_l1: mass 0.02 -> 1; geometry visual box size=0 0 0
- link _ring_proximal_l0: mass 0.03 -> 0.01; geometry visual box size=0 0 0
- link _ring_proximal_l1: mass 0.02 -> 1; geometry visual box size=0 0 0
- link _thumb_chassis_l0: mass 0.03 -> 0.01; geometry visual box size=0 0 0
- link _thumb_chassis_l1: mass 0.02 -> 1; geometry visual box size=0 0 0
- link _thumb_distal_l0: mass 0.03 -> 0.01; geometry visual box size=0 0 0
- link _thumb_distal_l1: mass 0.02 -> 1; geometry visual box size=0 0 0
- link _thumb_follower_l0: mass 0.03 -> 0.01; geometry visual box size=0 0 0
- link _thumb_follower_l1: mass 0.02 -> 1; geometry visual box size=0 0 0
- link _thumb_link_l0: mass 0.03 -> 0.01; geometry visual box size=0 0 0
- link _thumb_link_l1: mass 0.02 -> 1; geometry visual box size=0 0 0
- link _thumb_proximal_l0: mass 0.03 -> 0.01; geometry visual box size=0 0 0
- link _thumb_proximal_l1: mass 0.02 -> 1; geometry visual box size=0 0 0
- link base_link: mass 0.35 -> 0.5; geometry collision box size=0.08 0.08 0.08; visual mesh filename=package://hand_pack/urdf/linear_meshes/right_base_link.STL scale=0.0625 0.0625 0.0625
- link index_distal: mass 0.015 -> 0.01
- link index_follower: mass 0.015 -> 0.01
- link index_knuckle: mass 0.015 -> 0.01
- link index_link: mass 0.015 -> 0.01
- link index_proximal: mass 0.015 -> 0.01
- link lisa: mass 0.005 -> 0.01
- link little_distal: mass 0.015 -> 0.01
- link little_follower: mass 0.015 -> 0.01
- link little_knuckle: mass 0.015 -> 0.01
- link little_link: mass 0.015 -> 0.01
- link little_proximal: mass 0.015 -> 0.01
- link middle_distal: mass 0.015 -> 0.01
- link middle_follower: mass 0.015 -> 0.01
- link middle_knuckle: mass 0.015 -> 0.01
- link middle_link: mass 0.015 -> 0.01
- link middle_proximal: mass 0.015 -> 0.01
- link ring_distal: mass 0.015 -> 0.01
- link ring_follower: mass 0.015 -> 0.01
- link ring_knuckle: mass 0.015 -> 0.01
- link ring_link: mass 0.015 -> 0.01
- link ring_proximal: mass 0.015 -> 0.01
- link thumb_chassis: mass 0.015 -> 0.01
- link thumb_distal: mass 0.015 -> 0.01
- link thumb_follower: mass 0.015 -> 0.01
- link thumb_link: mass 0.015 -> 0.01
- link thumb_proximal: mass 0.015 -> 0.01
Joints:
- removed joint __joint_base_link
- removed joint _joint_base_link
- added joint base_joint: type fixed, parent base_footprint, child base_link, origin xyz=0 0 0.1
- joint Index: limit lower=0.00000000000000000000 upper=1.00000000000000000000 effort=0 velocity=0 -> lower=0.00000000000000000000 upper=1.00000000000000000000 effort=10.0 velocity=1.0
- joint Little: limit lower=0.00000000000000000000 upper=1.00000000000000000000 effort=0 velocity=0 -> lower=0.00000000000000000000 upper=1.00000000000000000000 effort=10.0 velocity=1.0
- joint Middle: limit lower=0.00000000000000000000 upper=1.00000000000000000000 effort=0 velocity=0 -> lower=0.00000000000000000000 upper=1.00000000000000000000 effort=10.0 velocity=1.0
- joint Ring: limit lower=0.00000000000000000000 upper=1.00000000000000000000 effort=0 velocity=0 -> lower=0.00000000000000000000 upper=1.00000000000000000000 effort=10.0 velocity=1.0
- joint Rotate: limit lower=0.00000000000000000000 upper=1.00000000000000000000 effort=0 velocity=0 -> lower=0.00000000000000000000 upper=1.00000000000000000000 effort=10.0 velocity=1.0
- joint Thumb: limit lower=0.00000000000000000000 upper=1.00000000000000000000 effort=0 velocity=0 -> lower=0.00000000000000000000 upper=1.00000000000000000000 effort=10.0 velocity=1.0
- joint _index_distal_j01: limit lower=0.00000002107342395030 upper=1.33574110944277979485 effort=0 velocity=0 -> lower=0.00000002107342395030 upper=1.33574110944277979485 effort=10.0 velocity=1.0
- joint _index_follower_j01: limit lower=-0.00000000000000005551 upper=0.26422627443923901724 effort=0 velocity=0 -> lower=-0.00000000000000005551 upper=0.26422627443923901724 effort=10.0 velocity=1.0
- joint _index_knuckle_j01: limit lower=0.00000002107342400581 upper=1.25181521906792703192 effort=0 velocity=0 -> lower=0.00000002107342400581 upper=1.25181521906792703192 effort=10.0 velocity=1.0
- joint _index_link_j01: limit lower=-0.00000000000000033307 upper=1.33574038782547499515 effort=0 velocity=0 -> lower=-0.00000000000000033307 upper=1.33574038782547499515 effort=10.0 velocity=1.0
- joint _index_proximal_j01: limit lower=0.00000001490116086078 upper=1.51604341403629772067 effort=0 velocity=0 -> lower=0.00000001490116086078 upper=1.51604341403629772067 effort=10.0 velocity=1.0
- joint _lisa_j01: limit lower=0.00000001490116097180 upper=1.07337743464992829701 effort=0 velocity=0 -> lower=0.00000001490116097180 upper=1.07337743464992829701 effort=10.0 velocity=1.0
- joint _little_distal_j01: limit lower=0.00000001490116086078 upper=1.31664154360936347388 effort=0 velocity=0 -> lower=0.00000001490116086078 upper=1.31664154360936347388 effort=10.0 velocity=1.0
- joint _little_follower_j01: limit lower=-0.00000000000000005551 upper=0.26422625333146310123 effort=0 velocity=0 -> lower=-0.00000000000000005551 upper=0.26422625333146310123 effort=10.0 velocity=1.0
- joint _little_knuckle_j01: limit lower=0.00000001490116097180 upper=1.25181530552105346743 effort=0 velocity=0 -> lower=0.00000001490116097180 upper=1.25181530552105346743 effort=10.0 velocity=1.0
- joint _little_link_j01: limit lower=-0.00000000000000022204 upper=1.31664159359669952210 effort=0 velocity=0 -> lower=-0.00000000000000022204 upper=1.31664159359669952210 effort=10.0 velocity=1.0
- joint _little_proximal_j01: limit lower=-0.00000000000000022204 upper=1.51604353824540583062 effort=0 velocity=0 -> lower=-0.00000000000000022204 upper=1.51604353824540583062 effort=10.0 velocity=1.0
- joint _middle_distal_j01: limit lower=0.00000002107342389479 upper=1.34986013639683699594 effort=0 velocity=0 -> lower=0.00000002107342389479 upper=1.34986013639683699594 effort=10.0 velocity=1.0
- joint _middle_follower_j01: limit lower=-0.00000000000000005551 upper=0.26422641895880316643 effort=0 velocity=0 -> lower=-0.00000000000000005551 upper=0.26422641895880316643 effort=10.0 velocity=1.0
- joint _middle_knuckle_j01: limit lower=-0.00000000000000022204 upper=1.25181499257524886382 effort=0 velocity=0 -> lower=-0.00000000000000022204 upper=1.25181499257524886382 effort=10.0 velocity=1.0
- joint _middle_link_j01: limit lower=-0.00000000000000027756 upper=1.34986028913700639720 effort=0 velocity=0 -> lower=-0.00000000000000027756 upper=1.34986028913700639720 effort=10.0 velocity=1.0
- joint _middle_proximal_j01: limit lower=-0.00000000000000055511 upper=1.51604368978712988891 effort=0 velocity=0 -> lower=-0.00000000000000055511 upper=1.51604368978712988891 effort=10.0 velocity=1.0
- joint _ring_distal_j01: limit lower=-0.00000000000000033307 upper=1.34878317629562749502 effort=0 velocity=0 -> lower=-0.00000000000000033307 upper=1.34878317629562749502 effort=10.0 velocity=1.0
- joint _ring_follower_j01: limit lower=-0.00000000000000005551 upper=0.26423062522385393214 effort=0 velocity=0 -> lower=-0.00000000000000005551 upper=0.26423062522385393214 effort=10.0 velocity=1.0
- joint _ring_knuckle_j01: limit lower=-0.00000000000000033307 upper=1.25181510906761417345 effort=0 velocity=0 -> lower=-0.00000000000000033307 upper=1.25181510906761417345 effort=10.0 velocity=1.0
- joint _ring_link_j01: limit lower=-0.00000000000000027756 upper=1.34878364034376607705 effort=0 velocity=0 -> lower=-0.00000000000000027756 upper=1.34878364034376607705 effort=10.0 velocity=1.0
- joint _ring_proximal_j01: limit lower=-0.00000000000000022204 upper=1.51604328762193540925 effort=0 velocity=0 -> lower=-0.00000000000000022204 upper=1.51604328762193540925 effort=10.0 velocity=1.0
- joint _thumb_chassis_j01: limit lower=0.00000002107342389479 upper=1.53339620392031616980 effort=0 velocity=0 -> lower=0.00000002107342389479 upper=1.53339620392031616980 effort=10.0 velocity=1.0
- joint _thumb_distal_j01: limit lower=-0.00000000000000033307 upper=1.06686018440504426508 effort=0 velocity=0 -> lower=-0.00000000000000033307 upper=1.06686018440504426508 effort=10.0 velocity=1.0
- joint _thumb_follower_j01: limit lower=-0.00000000000000022204 upper=0.93732763826281428887 effort=0 velocity=0 -> lower=-0.00000000000000022204 upper=0.93732763826281428887 effort=10.0 velocity=1.0
- joint _thumb_link_j01: limit lower=-0.00000000000000016653 upper=0.76799454671461697686 effort=0 velocity=0 -> lower=-0.00000000000000016653 upper=0.76799454671461697686 effort=10.0 velocity=1.0
- joint _thumb_proximal_j01: limit lower=-0.00000000000000016653 upper=0.72022188617106019937 effort=0 velocity=0 -> lower=-0.00000000000000016653 upper=0.72022188617106019937 effort=10.0 velocity=1.0
- joint world_fixed: child __base_link -> base_footprint; origin xyz=0 0 0.1 rpy=0 0 0 -> (none)

Commit message: pronto para iniciar o controle

File: install/hand_pack/share/hand_pack/urdf/linear_covvi_hand_gazebo.urdf (robot description, URDF)
Before this commit: robot covvi_digital_twin_perfect, 87 links, 86 joints
Joints:
- joint _index_link_j01: type revolute -> fixed
- joint _little_link_j01: type revolute -> fixed
- joint _middle_link_j01: type revolute -> fixed
- joint _ring_link_j01: type revolute -> fixed

File: src/hand_pack/urdf/invisible_mech_covvi_hand.urdf (robot description, URDF)
Before this commit: robot covvi_digital_twin_perfect, 87 links, 86 joints
Joints:
- joint _index_link_j01: type fixed -> revolute
- joint _little_link_j01: type fixed -> revolute
- joint _middle_link_j01: type fixed -> revolute
- joint _ring_link_j01: type fixed -> revolute
