Commit message: adicionado novo effector

File: src/cra_description/urdf/cr10_robot.xacro (robot description, xacro)
@@ -27,5 +27,5 @@
         name="">
         <color
-          rgba="1 1 1 1" />
+          rgba="0.20 0.20 0.22 1" />
       </material>
     </visual>
@@ -77,5 +77,5 @@
         name="">
         <color
-          rgba="1 1 1 1" />
+          rgba="0.20 0.20 0.22 1" />
       </material>
     </visual>
@@ -135,5 +135,5 @@
         name="">
         <color
-          rgba="1 1 1 1" />
+          rgba="0.72 0.72 0.75 1" />
       </material>
     </visual>
@@ -193,5 +193,5 @@
         name="">
         <color
-          rgba="1 1 1 1" />
+          rgba="0.72 0.72 0.75 1" />
       </material>
     </visual>
@@ -251,5 +251,5 @@
         name="">
         <color
-          rgba="1 1 1 1" />
+          rgba="0.20 0.20 0.22 1" />
       </material>
     </visual>
@@ -309,5 +309,5 @@
         name="">
         <color
-          rgba="1 1 1 1" />
+          rgba="0.20 0.20 0.22 1" />
       </material>
     </visual>
@@ -367,5 +367,5 @@
         name="">
         <color
-          rgba="1 1 1 1" />
+          rgba="0.84 0.84 0.86 1" />
       </material>
     </visual>
@@ -401,28 +401,35 @@
         <gravity>false</gravity>
         <selfCollide>true</selfCollide>
+        <visual><material><ambient>0.20 0.20 0.22 1</ambient><diffuse>0.20 0.20 0.22 1</diffuse><specular>0.35 0.35 0.38 1</specular></material></visual>
     </gazebo>
     <gazebo reference="Link1">
         <gravity>false</gravity>
         <selfCollide>true</selfCollide>
+        <visual><material><ambient>0.20 0.20 0.22 1</ambient><diffuse>0.20 0.20 0.22 1</diffuse><specular>0.35 0.35 0.38 1</specular></material></visual>
     </gazebo>
     <gazebo reference="Link2">
         <gravity>false</gravity>
         <selfCollide>true</selfCollide>
+        <visual><material><ambient>0.72 0.72 0.75 1</ambient><diffuse>0.72 0.72 0.75 1</diffuse><specular>0.6 0.6 0.65 1</specular></material></visual>
     </gazebo>
     <gazebo reference="Link3">
         <gravity>false</gravity>
         <selfCollide>true</selfCollide>
+        <visual><material><ambient>0.72 0.72 0.75 1</ambient><diffuse>0.72 0.72 0.75 1</diffuse><specular>0.6 0.6 0.65 1</specular></material></visual>
     </gazebo>
     <gazebo reference="Link4">
         <gravity>false</gravity>
         <selfCollide>true</selfCollide>
+        <visual><material><ambient>0.20 0.20 0.22 1</ambient><diffuse>0.20 0.20 0.22 1</diffuse><specular>0.35 0.35 0.38 1</specular></material></visual>
     </gazebo>
     <gazebo reference="Link5">
         <gravity>false</gravity>
         <selfCollide>true</selfCollide>
+        <visual><material><ambient>0.20 0.20 0.22 1</ambient><diffuse>0.20 0.20 0.22 1</diffuse><specular>0.35 0.35 0.38 1</specular></material></visual>
     </gazebo>
     <gazebo reference="Link6">
         <gravity>false</gravity>
         <selfCollide>true</selfCollide>
+        <visual><material><ambient>0.84 0.84 0.86 1</ambient><diffuse>0.84 0.84 0.86 1</diffuse><specular>0.7 0.7 0.72 1</specular></material></visual>
     </gazebo>
     <!-- 在运行demo.launch.py时，需要注释这个ros2_control节点，因为它使用了xxx.ros2_control.xacro来生成了ros2_control节点-->

Commit message: real arm

File: src/cra_description/urdf/cr10_robot.xacro (robot description, xacro)
@@ -1,507 +1,570 @@
 <?xml version="1.0"?>
 <robot name="cr10_robot" xmlns:xacro="http://ros.org/wiki/xacro">
+  <!-- ========================================================
+       CR10A — 6 joints, 6 blue accent rings (one per joint)
+       Ring placement: child of the CHILD link, at the shaft
+       neck visible at each joint interface.
+       ======================================================== -->
   <link name="dummy_link"/>
+  <!-- ===== base_link ===== -->
   <link name="base_link">
     <inertial>
-      <origin
-        xyz="-0.0017435 -4.7141E-06 0.032774" rpy="0 0 0" />
-      <mass
-        value="1.8265" />
-      <inertia
-        ixx="0.0041731"
-        ixy="5.9354E-07"
-        ixz="2.52E-05"
-        iyy="0.0043128"
-        iyz="-5.4503E-07"
-        izz="0.0067702" />
-    </inertial>
-    <visual>
-      <origin
-        xyz="0 0 0"
-        rpy="0 0 0" />
-      <geometry>
-        <mesh
-          filename="file://$(find cra_description)/meshes/cr10/base_link.STL" />
-      </geometry>
-      <material
-        name="">
-        <color
-          rgba="0.20 0.20 0.22 1" />
-      </material>
-    </visual>
-    <collision>
-      <origin
-        xyz="0 0 0"
-        rpy="0 0 0" />
-      <geometry>
-        <mesh
-          filename="file://$(find cra_description)/meshes/cr10/base_link.STL" />
-      </geometry>
-    </collision>
-  </link>
-  <link  name="world"/>
-<joint name="world_joint" type="fixed">
+      <origin xyz="-0.0017435 -4.7141E-06 0.032774" rpy="0 0 0" />
+      <mass value="1.8265" />
+      <inertia ixx="0.0041731" ixy="5.9354E-07" ixz="2.52E-05"
+               iyy="0.0043128" iyz="-5.4503E-07" izz="0.0067702" />
+    </inertial>
+    <visual>
+      <origin xyz="0 0 0" rpy="0 0 0"/>
+      <geometry><mesh filename="file://$(find cra_description)/meshes/cr10/base_link.STL"/></geometry>
+      <material name="body_gray"><color rgba="0.800 0.800 0.800 1"/></material>
+    </visual>
+    <collision>
+      <origin xyz="0 0 0" rpy="0 0 0"/>
+      <geometry><mesh filename="file://$(find cra_description)/meshes/cr10/base_link.STL"/></geometry>
+    </collision>
+  </link>
+  <link name="world"/>
+  <joint name="world_joint" type="fixed">
     <origin xyz="0 0 0.03" rpy="0 0 0" />
     <parent link="world" />
-    <child  link="dummy_link" />
+    <child link="dummy_link" />
   </joint>
   <joint name="dummy_joint" type="fixed">
     <parent link="dummy_link" />
-    <child  link="base_link" />
-  </joint>
-  <link
-    name="Link1">
-    <inertial>
-      <origin
-        xyz="-1.6635E-06 -0.010819 0.0028389"
-        rpy="0 0 0" />
-      <mass
-        value="4.1649" />
-      <inertia
-        ixx="0.020714"
-        ixy="-1.9343E-07"
-        ixz="1.6036E-07"
-        iyy="0.018824"
-        iyz="-9.6731E-05"
-        izz="0.014575" />
-    </inertial>
-    <visual>
-      <origin
-        xyz="0 0 0"
-        rpy="0 0 0" />
+    <child link="base_link" />
+  </joint>
+  <!-- ===== Link1 — shoulder housing ===== -->
+  <!-- Link1 mesh neck radii:
+         Z=-0.083 (joint1 groove): r_max=0.077 m
+         Z=+0.087 (joint2 groove): r_max=0.073 m               -->
+  <link name="Link1">
+    <inertial>
+      <origin xyz="-1.6635E-06 -0.010819 0.0028389" rpy="0 0 0" />
+      <mass value="4.1649" />
+      <inertia ixx="0.020714" ixy="-1.9343E-07" ixz="1.6036E-07"
+               iyy="0.018824" iyz="-9.6731E-05" izz="0.014575" />
+    </inertial>
+    <visual>
+      <origin xyz="0 0 0" rpy="0 0 0" />
+      <geometry><mesh filename="file://$(find cra_description)/meshes/cr10/Link1.STL"/></geometry>
+      <material name="body_gray"><color rgba="0.800 0.800 0.800 1"/></material>
+    </visual>
+    <collision>
+      <origin xyz="0 0 0" rpy="0 0 0"/>
+      <geometry><mesh filename="file://$(find cra_description)/meshes/cr10/Link1.STL"/></geometry>
+    </collision>
+  </link>
+  <joint name="joint1" type="revolute">
+    <origin xyz="0 0 0.1765" rpy="0 0 0" />
+    <parent link="base_link" />
+    <child link="Link1" />
+    <axis xyz="0 0 -1" />
+    <limit lower="-6.27" upper="6.27" effort="300" velocity="100" />
+  </joint>
+  <!-- JOINT 1 ring — at the bottom neck of Link1 shoulder housing (Z=-0.083).
+       Mesh outer radius at this section = 0.077 m → ring at 0.083 m             -->
+  <link name="ring_j1">
+    <visual>
+      <origin xyz="0 0 0" rpy="0 0 0"/>
+      <geometry><cylinder radius="0.0830" length="0.0140"/></geometry>
+      <material name="dobot_blue"><color rgba="0.157 0.290 0.690 1"/></material>
+    </visual>
+  </link>
+  <joint name="joint_ring_j1" type="fixed">
+    <origin xyz="0 0 -0.0830" rpy="0 0 0"/>
+    <parent link="Link1"/>
+    <child link="ring_j1"/>
+  </joint>
+  <link name="cap_j1">
+    <visual>
+      <origin xyz="0 0 0" rpy="0 0 0"/>
+      <geometry><cylinder radius="0.0890" length="0.0060"/></geometry>
+      <material name="joint_white"><color rgba="0.900 0.900 0.900 1"/></material>
+    </visual>
+  </link>
+  <joint name="joint_cap_j1" type="fixed">
+    <origin xyz="0 0 -0.0760" rpy="0 0 0"/>
+    <parent link="Link1"/>
+    <child link="cap_j1"/>
+  </joint>
+  <!-- JOINT 2 ring — at the top neck of Link1 shoulder housing (Z=+0.087).
+       Mesh outer radius at this section = 0.073 m → ring at 0.079 m             -->
+  <link name="ring_j2">
+    <visual>
+      <origin xyz="0 0 0" rpy="0 0 0"/>
+      <geometry><cylinder radius="0.0790" length="0.0140"/></geometry>
+      <material name="dobot_blue"><color rgba="0.157 0.290 0.690 1"/></material>
+    </visual>
+  </link>
+  <joint name="joint_ring_j2" type="fixed">
+    <origin xyz="0 0 0.0870" rpy="0 0 0"/>
+    <parent link="Link1"/>
+    <child link="ring_j2"/>
+  </joint>
+  <link name="cap_j2">
+    <visual>
+      <origin xyz="0 0 0" rpy="0 0 0"/>
+      <geometry><cylinder radius="0.0850" length="0.0060"/></geometry>
+      <material name="joint_white"><color rgba="0.900 0.900 0.900 1"/></material>
+    </visual>
+  </link>
+  <joint name="joint_cap_j2" type="fixed">
+    <origin xyz="0 0 0.0810" rpy="0 0 0"/>
+    <parent link="Link1"/>
+    <child link="cap_j2"/>
+  </joint>
+  <!-- ===== Link2 — upper arm ===== -->
+  <!-- Link2 arm tube runs along X. Tube center is offset Z=+0.193 from link origin.
+       Joint3 is at X=-0.607 in Link2 frame. Ring placed at the end of the arm tube
+       (X=-0.555, Z=0.193) just before the elbow housing begins.                  -->
+  <link name="Link2"><!-- joint1 keeps axis -1 -->
+    <inertial>
+      <origin xyz="-0.24631 3.5816E-07 0.19515" rpy="0 0 0" />
+      <mass value="11.314" />
+      <inertia ixx="0.033616" ixy="-8.2998E-07" ixz="-0.0033352"
+               iyy="0.30683" iyz="-6.6457E-08" izz="0.29972" />
+    </inertial>
+    <visual>
+      <origin xyz="0 0 0" rpy="0 0 0" />
       <geometry>
-        <mesh
-          filename="file://$(find cra_description)/meshes/cr10/Link1.STL" />
+        <mesh filename="file://$(find cra_description)/meshes/cr10/Link2.STL"  />
       </geometry>
-      <material
-        name="">
-        <color
-          rgba="0.20 0.20 0.22 1" />
-      </material>
-    </visual>
-    <collision>
-      <origin
-        xyz="0 0 0"
-        rpy="0 0 0" />
+      <material name="body_gray"><color rgba="0.800 0.800 0.800 1"/></material>
+    </visual>
+    <collision>
+      <origin xyz="0 0 0" rpy="0 0 0"/>
+      <geometry><mesh filename="file://$(find cra_description)/meshes/cr10/Link2.STL"/></geometry>
+    </collision>
+  </link>
+  <joint name="joint2" type="revolute">
+    <origin xyz="0 0 0" rpy="1.5708 1.5708 0" />
+    <parent link="Link1" />
+    <child link="Link2" />
+    <axis xyz="0 0 1" />
+    <limit lower="-6.27" upper="6.27" effort="300" velocity="100" />
+  </joint>
+  <!-- JOINT 3 ring — at elbow end of Link2 arm tube.
+       Arm tube center at X=-0.555: (Y=0, Z=0.193). Tube r≈60 mm → ring at 70 mm.
+       Cylinder axis along X (rpy 0 π/2 0).                                       -->
+  <link name="ring_j3">
+    <visual>
+      <origin xyz="0 0 0" rpy="0 1.5708 0"/>
+      <geometry><cylinder radius="0.0700" length="0.0140"/></geometry>
+      <material name="dobot_blue"><color rgba="0.157 0.290 0.690 1"/></material>
+    </visual>
+  </link>
+  <joint name="joint_ring_j3" type="fixed">
+    <origin xyz="-0.5550 0 0.1930" rpy="0 0 0"/>
+    <parent link="Link2"/>
+    <child link="ring_j3"/>
+  </joint>
+  <link name="cap_j3">
+    <visual>
+      <origin xyz="0 0 0" rpy="0 1.5708 0"/>
+      <geometry><cylinder radius="0.0760" length="0.0060"/></geometry>
+      <material name="joint_white"><color rgba="0.900 0.900 0.900 1"/></material>
+    </visual>
+  </link>
+  <joint name="joint_cap_j3" type="fixed">
+    <origin xyz="-0.5490 0 0.1930" rpy="0 0 0"/>
+    <parent link="Link2"/>
+    <child link="cap_j3"/>
+  </joint>
+  <!-- ===== Link3 — forearm ===== -->
+  <link name="Link3">
+    <inertial>
+      <origin xyz="-0.270855859955203 2.5144690851208E-07 0.0622960395387155" rpy="0 0 0" />
+      <mass value="4.89191189064363" />
+      <inertia ixx="0.00715720724136357" ixy="-5.62017408817872E-07" ixz="-0.00257748068989916"
+               iyy="0.239673426443838" iyz="9.26228295895878E-08" izz="0.238369168055991" />
+    </inertial>
+    <visual>
+      <origin xyz="0 0 0" rpy="0 0 0" />
       <geometry>
-        <mesh
-          filename="file://$(find cra_description)/meshes/cr10/Link1.STL" />
+        <mesh filename="file://$(find cra_description)/meshes/cr10/Link3.STL"  />
       </geometry>
-    </collision>
-  </link>
-  <joint
-    name="joint1"
-    type="revolute">
-    <origin
-      xyz="0 0 0.1765"
-      rpy="0 0 0" />
-    <parent
-      link="base_link" />
-    <child
-      link="Link1" />
-    <axis
-      xyz="0 0 -1" />
-    <limit
-      lower="-6.27"
-      upper="6.27"
-      effort="300"
-      velocity="100" />
-  </joint>
-  <link
-    name="Link2"><!-- joint1 keeps axis -1 (CR10 j1 rotates CW-positive, opposite of +Z) -->
-    <inertial>
-      <origin
-        xyz="-0.24631 3.5816E-07 0.19515"
-        rpy="0 0 0" />
-      <mass
-        value="11.314" />
-      <inertia
-        ixx="0.033616"
-        ixy="-8.2998E-07"
-        ixz="-0.0033352"
-        iyy="0.30683"
-        iyz="-6.6457E-08"
-        izz="0.29972" />
-    </inertial>
-    <visual>
-      <origin
-        xyz="0 0 0"
-        rpy="0 0 0" />
+      <material name="body_gray"><color rgba="0.800 0.800 0.800 1"/></material>
+    </visual>
+    <collision>
+      <origin xyz="0 0 0" rpy="0 0 0"/>
+      <geometry><mesh filename="file://$(find cra_description)/meshes/cr10/Link3.STL"/></geometry>
+    </collision>
+  </link>
+  <joint name="joint3" type="revolute">
+    <origin xyz="-0.607 0 0" rpy="0 0 0" />
+    <parent link="Link2" />
+    <child link="Link3" />
+    <axis xyz="0 0 1" />
+    <limit lower="-2.861" upper="2.861" effort="300" velocity="100" />
+  </joint>
+  <!-- ===== Link4 — wrist roll ===== -->
+  <!-- Link4 bottom neck (joint4 shaft entry) at Z=-0.060.
+       Mesh r_max at neck = 0.046 m → ring at 0.053 m                            -->
+  <link name="Link4">
+    <inertial>
+      <origin xyz="-2.53137491438456E-07 0.00798724498566683 -0.00589074229668524" rpy="0 0 0" />
+      <mass value="1.16884294495796" />
+      <inertia ixx="0.00292614933092813" ixy="8.20440076221281E-09" ixz="-8.19990423351321E-09"
+               iyy="0.00150052997722543" iyz="-5.4492521866877E-05" izz="0.00273274943535585" />
+    </inertial>
+    <visual>
+      <origin xyz="0 0 0" rpy="0 0 0" />
       <geometry>
-        <mesh
-          filename="file://$(find cra_description)/meshes/cr10/Link2.STL"  />
+        <mesh filename="file://$(find cra_description)/meshes/cr10/Link4.STL"/>
       </geometry>
-      <material
-        name="">
-        <color
-          rgba="0.72 0.72 0.75 1" />
-      </material>
-    </visual>
-    <collision>
-      <origin
-        xyz="0 0 0"
-        rpy="0 0 0" />
+      <material name="body_gray"><color rgba="0.800 0.800 0.800 1"/></material>
+    </visual>
+    <collision>
+      <origin xyz="0 0 0" rpy="0 0 0"/>
+      <geometry><mesh filename="file://$(find cra_description)/meshes/cr10/Link4.STL"/></geometry>
+    </collision>
+  </link>
+  <joint name="joint4" type="revolute">
+    <origin xyz="-0.568 0 0.191" rpy="0 0 -1.5708" />
+    <parent link="Link3" />
+    <child link="Link4" />
+    <axis xyz="0 0 1" />
+    <limit lower="-6.27" upper="6.27" effort="300" velocity="100" />
+  </joint>
+  <!-- JOINT 4 ring — bottom neck of Link4 (where the joint4 shaft enters the wrist housing) -->
+  <link name="ring_j4">
+    <visual>
+      <origin xyz="0 0 0" rpy="0 0 0"/>
+      <geometry><cylinder radius="0.0530" length="0.0130"/></geometry>
+      <material name="dobot_blue"><color rgba="0.157 0.290 0.690 1"/></material>
+    </visual>
+  </link>
+  <joint name="joint_ring_j4" type="fixed">
+    <origin xyz="0 0 -0.0600" rpy="0 0 0"/>
+    <parent link="Link4"/>
+    <child link="ring_j4"/>
+  </joint>
+  <link name="cap_j4">
+    <visual>
+      <origin xyz="0 0 0" rpy="0 0 0"/>
+      <geometry><cylinder radius="0.0590" length="0.0060"/></geometry>
+      <material name="joint_white"><color rgba="0.900 0.900 0.900 1"/></material>
+    </visual>
+  </link>
+  <joint name="joint_cap_j4" type="fixed">
+    <origin xyz="0 0 -0.0530" rpy="0 0 0"/>
+    <parent link="Link4"/>
+    <child link="cap_j4"/>
+  </joint>
+  <!-- ===== Link5 — wrist pitch ===== -->
+  <!-- Link5 bottom neck at Z=-0.057. Mesh r_max = 0.046 m → ring at 0.053 m    -->
+  <link name="Link5">
+    <inertial>
+      <origin xyz="5.50699455951951E-07 -0.0145467578029201 -0.00454887087411437" rpy="0 0 0" />
+      <mass value="1.22303084244711" />
+      <inertia ixx="0.00337905462069531" ixy="3.57819902464362E-08" ixz="-7.51828060542842E-09"
+               iyy="0.00149255573951137" iyz="8.41917918947542E-05" izz="0.00323300312341709" />
+    </inertial>
+    <visual>
+      <origin xyz="0 0 0" rpy="0 0 0" />
       <geometry>
-        <mesh
-          filename="file://$(find cra_description)/meshes/cr10/Link2.STL" />
+        <mesh filename="file://$(find cra_description)/meshes/cr10/Link5.STL" />
       </geometry>
-    </collision>
-  </link>
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