Commit message: testes

File: src/touch_pack/urdf/touch_tool_square_20x20.urdf (robot description, URDF)
Before this commit: robot touch_tool_tcp, 4 links, 3 joints
Links:
- added link force_sensor_link, mass 0.150; collision box size=0.0508 0.0127 0.060; visual mesh filename=package://touch_pack/meshes/Celula De Carga.stl scale=0.001 0.001 0.001
Joints:
- added joint force_sensor_attach: type fixed, parent Link6, child force_sensor_link, origin xyz=0 0 0 rpy=0 0 0
- joint touch_tool_attach: origin xyz=0 0 0 rpy=0 0 0 -> xyz=0 0 0.060 rpy=0 0 0; parent Link6 -> force_sensor_link

Commit message: software de poses

File: src/touch_pack/urdf/touch_tool_square_20x20.urdf (robot description, URDF)
Before this commit: robot touch_tool_tcp, 5 links, 4 joints
Links:
- added link lower_coupling_link, mass 0.200; collision cylinder length=0.015 radius=0.040; visual mesh filename=package://touch_pack/meshes/Acoplador_CelulaDeCarga_Uniaxia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 scale=0.001 0.001 0.001
- added link upper_coupling_link, mass 0.200; collision cylinder length=0.015 radius=0.040; visual mesh filename=package://touch_pack/meshes/Acoplador_CelulaDeCarga_Uniaxia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 scale=0.001 0.001 0.001
Joints:
- added joint lower_coupling_attach: type fixed, parent Link6, child lower_coupling_link, origin xyz=0 0 0 rpy=0 0 0
- added joint upper_coupling_attach: type fixed, parent force_sensor_link, child upper_coupling_link, origin xyz=0 0 0.052 rpy=0 0 0
- joint force_sensor_attach: origin xyz=0 0 0 rpy=0 0 0 -> xyz=0 0 0.007 rpy=0 0 0; parent Link6 -> lower_coupling_link
- joint touch_tool_attach: origin xyz=0 0 0.060 rpy=0 0 0 -> xyz=0 0 0.015 rpy=0 0 0; parent force_sensor_link -> upper_coupling_link

Commit message: att

File: src/touch_pack/urdf/touch_tool_square_20x20.urdf (robot description, URDF)
Before this commit: robot touch_tool_tcp, 7 links, 6 joints
Links:
- removed link lower_coupling_link
- removed link upper_coupling_link
- link force_sensor_link: mass 0.150 -> 0.400; geometry collision box size=0.081 0.0127 0.0127; collision cylinder length=0.008 radius=0.035
Joints:
- removed joint lower_coupling_attach
- removed joint upper_coupling_attach
- joint force_sensor_attach: origin xyz=0 0 0.007 rpy=0 0 0 -> xyz=0 0 0 rpy=0 0 -1.5708; parent lower_coupling_link -> Link6
- joint touch_tool_attach: origin xyz=0 0 0.015 rpy=0 0 0 -> xyz=0.055 0 0.028 rpy=0 0 1.5708; parent upper_coupling_link -> force_sensor_link
